File: src/hardware/fc/_autosave-drone.kicad_pcb (KiCad board)
At the start: 4 copper layers, 40 x 40 mm, 121 parts, among them J1 Conn_01x01, J10 Conn_01x01, J11 Conn_01x01, J12 Conn_01x01, J13 Conn_01x01, J14 Conn_01x01, J15 Conn_01x01, J16 Conn_01x01, J17 Conn_01x01, J18 Conn_01x01, J19 Conn_01x03, J2 Conn_01x08, J20 Conn_01x03, J21 Conn_01x03, J22 Conn_01x03, J23 Conn_01x01, J24 Conn_01x01, J25 Conn_01x01, J3 Conn_01x01, J4 Conn_01x01, J5 Conn_01x01, J6 Conn_01x01, J7 Conn_01x01, J8 Conn_01x01, J9 Conn_01x01, Q1 AO3400A, Q2 NPN, Q3 NPN, SW1 SW_Push, SW2 SW_Push, U10 LM66100DCKR, U2 TLV75533PDBVR, U3 W25Q128JVSIQTR, U4 STM32F405RGTx, U5 ICM-42688-P, U6 LP5907MFX-3.3/NOPB, U7 AT7456E, U8 MP4420HGJ-Z, U9 LM66100DCKR, X1 XL2EL89CSI-111YLC-27M, Y1 C115962

Commit message: pcb update
Parts:
- removed C42, C43: 22uf, Capacitor_SMD:C_1206_3216Metric
- removed J12: Conn_01x01, footprint_lib:signal_pad
- removed R20: 150k, Resistor_SMD:R_0603_1608Metric
- removed R8: 41.2k, Resistor_SMD:R_0402_1005Metric
- removed U8: MP4420HGJ-Z, easyeda2kicad:TSOT-23-8_L2.9-W1.6-P0.65-LS2.8-BL
- added C44: 470nf, Capacitor_SMD:C_0603_1608Metric, B.Cu at (39.1, 37.5)
- added C45: 2.2uF, Capacitor_SMD:C_0402_1005Metric, B.Cu at (38.6, 35.2)
- added C46: 22uf, Capacitor_SMD:C_1206_3216Metric, B.Cu at (40.2, 42.5)
- added C47: 1uF, Capacitor_SMD:C_0402_1005Metric, B.Cu at (38.6, 34.2)
- added C48: 22pf, Capacitor_SMD:C_0402_1005Metric, B.Cu at (42.6, 33.2)
- added C50: 22uf, Capacitor_SMD:C_1206_3216Metric, B.Cu at (46.1, 38.2)
- added L2: 2.2uH, easyeda2kicad:IND-SMD_L4.8-W4.5, B.Cu at (34.9, 39.0)
- added R22: 17.8k, Resistor_SMD:R_0402_1005Metric, B.Cu at (40.6, 33.2)
- added R23: 1M, Resistor_SMD:R_0402_1005Metric, B.Cu at (45.6, 33.8)
- added R24: 127k, Resistor_SMD:R_0402_1005Metric, B.Cu at (46.9, 35.2)
- added U1: LM43603DSUR, easyeda2kicad:SON-16_L5.0-W4.0-P0.50-TL-EP, B.Cu at (53.0, 38.1)
- added U11: LM43603DSUR, easyeda2kicad:SON-16_L5.0-W4.0-P0.50-TL-EP, B.Cu at (42.5, 36.5)
- C16, D4, Q1, TP1, TP2: moved to B.Cu
- C17: value 100nf -> 22uf; footprint Capacitor_SMD:C_0402_1005Metric -> Capacitor_SMD:C_1206_3216Metric
- C18: value 100nf -> 22pf
- C19: value 22uf -> 470nf; footprint Capacitor_SMD:C_0805_2012Metric -> Capacitor_SMD:C_0603_1608Metric
- C20: value 100nf -> 2.2uF
- C37: value 22uf -> 1uF; footprint Capacitor_SMD:C_0805_2012Metric -> Capacitor_SMD:C_0402_1005Metric
- L1: value 1OuH -> 2.2uH; footprint Inductor_SMD:L_KOHERelec_MDA7030 -> easyeda2kicad:IND-SMD_L4.8-W4.5
- R5: value 20 -> 249k
- R6: value 7.68k -> 1M
- R7: value 51k -> 17.8k
- moved J1 65.6 mm to (39.8, 65.8)
- moved J3 63.5 mm to (44.8, 65.8)
- moved J14 60.7 mm to (42.2, 65.8)
- moved TP1 59.0 mm to (33.4, 58.5)
- moved TP2 59.0 mm to (36.2, 58.5)
- moved C16 56.2 mm to (31.5, 58.2), turned to -90 degrees
- moved J9 54.3 mm to (48.0, 65.8)
- moved J13 51.4 mm to (59.5, 65.8)
- moved Q1 50.7 mm to (39.2, 55.8), turned to 0 degrees
- moved J8 48.9 mm to (50.5, 65.8)
- moved J18 47.1 mm to (40.5, 32.2), turned to 180 degrees
- moved J17 42.7 mm to (42.8, 32.2), turned to 180 degrees
- moved J16 38.3 mm to (45.0, 32.2), turned to 180 degrees
- moved D4 37.2 mm to (34.8, 55.5), turned to 0 degrees
- moved J15 33.8 mm to (47.2, 32.2), turned to 180 degrees
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Connections:
- C17 pad 1: GND -> BAT_POWER_PROTECTED
- C17 pad 2: Net-(U8-VCC) -> GND
- C18 pad 1: Net-(U8-SW) -> Net-(U1-FB)
- C18 pad 2: Net-(C18-Pad2) -> LIPO_5V
- C19 pad 1: GND -> Net-(U1-CBOOT)
- C19 pad 2: LIPO_5V -> Net-(C19-Pad2)
- C20 pad 1: Net-(D6-K) -> Net-(U1-VCC)
- C31 pad 1: GND -> LIPO_5V
- C31 pad 2: Net-(D6-K) -> GND
- C37 pad 1: GND -> LIPO_5V
- C37 pad 2: LIPO_5V -> GND
- D6 pad 1: Net-(D6-K) -> BAT_POWER_PROTECTED
- D8 pad 1: Net-(D6-K) -> BAT_POWER_PROTECTED
- J6 pad 1: GND -> USART3_RX
- J7 pad 1: +5V -> USART3_TX
- J8 pad 1: RECEIVER_RX -> USART1_RX
- J9 pad 1: RECEIVER_TX -> USART1_TX
- L1 pad 1: Net-(U8-SW) -> Net-(C19-Pad2)
- R5 pad 1: Net-(U8-BST) -> Net-(U1-FB)
- R5 pad 2: Net-(C18-Pad2) -> GND
- R6 pad 1: Net-(R6-Pad1) -> LIPO_5V
- R6 pad 2: GND -> Net-(U1-FB)
- R7 pad 2: Net-(R6-Pad1) -> GND
- U4 pad 29: VTX_TX -> USART3_TX
- U4 pad 30: unconnected-(U4-PB11-Pad30) -> USART3_RX
- U4 pad 58: RECEIVER_RX -> USART1_TX
- U4 pad 59: RECEIVER_TX -> USART1_RX
Routing:
- net GND: track 0.00 -> 194.3 mm, vias 0 -> 65
- net VDD: track 0.00 -> 57.3 mm, vias 0 -> 11
- net +5V: track 0.00 -> 55.6 mm, vias 0 -> 12
- net +9V: track 0.00 -> 53.1 mm, vias 0 -> 2
- net BAT_POWER_PROTECTED: track 0.00 -> 37.3 mm
- net LIPO_5V: track 0.00 -> 33.8 mm
- net Net-(U10-ST): track 0.00 -> 28.8 mm, vias 0 -> 3
- net Net-(U10-~{CE}): track 0.00 -> 26.1 mm, vias 0 -> 3
- net PA6: track 0.00 -> 25.3 mm, vias 0 -> 2
- net PA5: track 0.00 -> 24.0 mm
- net PA7: track 0.00 -> 23.1 mm
- net BAT_CURR: track 0.00 -> 17.6 mm, vias 0 -> 1
- net VACC: track 0.00 -> 16.7 mm
- net Net-(U4-NRST): track 0.00 -> 14.5 mm
- net USB_D-: track 0.00 -> 13.8 mm
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- added copper zone on In2.Cu, net +5V
- added copper zone on In1.Cu, net GND
- added copper zone on In2.Cu, net VDD
- removed copper zone on In2.Cu, net GND
Other:
- board text added: "5v"
- board text added: "camera"
- board text added: "osd"
- board text added: "out"
- board text added: "uart(s1)"
- board text added: "uart(s3)"
- board text added: "vidin"
- board text removed: "lilex"
- board text removed: "uart"
