File: src/hardware/fc/drone.kicad_pcb (KiCad board)
At the start: 4 copper layers, 40 x 40 mm, 121 parts, among them J1 Conn_01x01, J10 Conn_01x01, J11 Conn_01x01, J12 Conn_01x01, J13 Conn_01x01, J14 Conn_01x01, J15 Conn_01x01, J16 Conn_01x01, J17 Conn_01x01, J18 Conn_01x01, J19 Conn_01x03, J2 Conn_01x08, J20 Conn_01x03, J21 Conn_01x03, J22 Conn_01x03, J23 Conn_01x01, J24 Conn_01x01, J25 Conn_01x01, J3 Conn_01x01, J4 Conn_01x01, J5 Conn_01x01, J6 Conn_01x01, J7 Conn_01x01, J8 Conn_01x01, J9 Conn_01x01, Q1 AO3400A, Q2 NPN, Q3 NPN, SW1 SW_Push, SW2 SW_Push, U10 LM66100DCKR, U2 TLV75533PDBVR, U3 W25Q128JVSIQTR, U4 STM32F405RGTx, U5 ICM-42688-P, U6 LP5907MFX-3.3/NOPB, U7 AT7456E, U8 MP4420HGJ-Z, U9 LM66100DCKR, X1 XL2EL89CSI-111YLC-27M, Y1 C115962

Commit message: pcb update
Parts:
- removed C42, C43: 22uf, Capacitor_SMD:C_1206_3216Metric
- removed J12: Conn_01x01, footprint_lib:signal_pad
- removed R20: 150k, Resistor_SMD:R_0603_1608Metric
- removed R8: 41.2k, Resistor_SMD:R_0402_1005Metric
- removed U8: MP4420HGJ-Z, easyeda2kicad:TSOT-23-8_L2.9-W1.6-P0.65-LS2.8-BL
- added C44: 470nf, Capacitor_SMD:C_0603_1608Metric, B.Cu at (39.1, 37.5)
- added C45: 2.2uF, Capacitor_SMD:C_0402_1005Metric, B.Cu at (38.6, 35.2)
- added C46: 22uf, Capacitor_SMD:C_1206_3216Metric, B.Cu at (40.2, 42.5)
- added C47: 1uF, Capacitor_SMD:C_0402_1005Metric, B.Cu at (38.6, 34.2)
- added C48: 22pf, Capacitor_SMD:C_0402_1005Metric, B.Cu at (42.6, 33.2)
- added C50: 22uf, Capacitor_SMD:C_1206_3216Metric, B.Cu at (46.1, 38.2)
- added L2: 2.2uH, easyeda2kicad:IND-SMD_L4.8-W4.5, B.Cu at (34.9, 39.0)
- added R22: 17.8k, Resistor_SMD:R_0402_1005Metric, B.Cu at (40.6, 33.2)
- added R23: 1M, Resistor_SMD:R_0402_1005Metric, B.Cu at (45.6, 33.8)
- added R24: 127k, Resistor_SMD:R_0402_1005Metric, B.Cu at (46.9, 35.2)
- added U1: LM43603DSUR, easyeda2kicad:SON-16_L5.0-W4.0-P0.50-TL-EP, B.Cu at (53.0, 38.1)
- added U11: LM43603DSUR, easyeda2kicad:SON-16_L5.0-W4.0-P0.50-TL-EP, B.Cu at (42.5, 36.5)
- C16, D4, Q1, TP1, TP2: moved to B.Cu
- C17: value 100nf -> 22uf; footprint Capacitor_SMD:C_0402_1005Metric -> Capacitor_SMD:C_1206_3216Metric
- C18: value 100nf -> 22pf
- C19: value 22uf -> 470nf; footprint Capacitor_SMD:C_0805_2012Metric -> Capacitor_SMD:C_0603_1608Metric
- C20: value 100nf -> 2.2uF
- C37: value 22uf -> 1uF; footprint Capacitor_SMD:C_0805_2012Metric -> Capacitor_SMD:C_0402_1005Metric
- L1: value 1OuH -> 2.2uH; footprint Inductor_SMD:L_KOHERelec_MDA7030 -> easyeda2kicad:IND-SMD_L4.8-W4.5
- R5: value 20 -> 249k
- R6: value 7.68k -> 1M
- R7: value 51k -> 17.8k
- moved J18 67.5 mm to (40.5, 32.2), turned to 180 degrees
- moved J1 65.6 mm to (39.8, 65.8)
- moved J3 63.5 mm to (44.8, 65.8)
- moved J17 62.8 mm to (42.8, 32.2), turned to 180 degrees
- moved J6 62.2 mm to (53.8, 65.8)
- moved J7 62.2 mm to (56.2, 65.8)
- moved J14 60.7 mm to (42.2, 65.8)
- moved J9 59.2 mm to (48.0, 65.8)
- moved J13 57.9 mm to (59.5, 65.8)
- moved C16 56.2 mm to (31.5, 58.2), turned to -90 degrees
- moved J5 55.5 mm to (49.5, 32.2), turned to 180 degrees
- moved J8 54.8 mm to (50.5, 65.8)
- moved J25 54.7 mm to (54.5, 32.8), turned to 180 degrees
- moved J15 53.4 mm to (47.2, 32.2), turned to 180 degrees
- moved J16 52.5 mm to (45.0, 32.2), turned to 180 degrees
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Connections:
- C17 pad 1: GND -> BAT_POWER_PROTECTED
- C17 pad 2: Net-(U8-VCC) -> GND
- C18 pad 1: Net-(U8-SW) -> Net-(U1-FB)
- C18 pad 2: Net-(C18-Pad2) -> LIPO_5V
- C19 pad 1: GND -> Net-(U1-CBOOT)
- C19 pad 2: LIPO_5V -> Net-(C19-Pad2)
- C20 pad 1: Net-(D6-K) -> Net-(U1-VCC)
- C31 pad 1: GND -> LIPO_5V
- C31 pad 2: Net-(D6-K) -> GND
- C37 pad 1: GND -> LIPO_5V
- C37 pad 2: LIPO_5V -> GND
- D6 pad 1: Net-(D6-K) -> BAT_POWER_PROTECTED
- D8 pad 1: Net-(D6-K) -> BAT_POWER_PROTECTED
- J6 pad 1: GND -> USART3_RX
- J7 pad 1: +5V -> USART3_TX
- J8 pad 1: RECEIVER_RX -> USART1_RX
- J9 pad 1: RECEIVER_TX -> USART1_TX
- L1 pad 1: Net-(U8-SW) -> Net-(C19-Pad2)
- R5 pad 1: Net-(U8-BST) -> Net-(U1-FB)
- R5 pad 2: Net-(C18-Pad2) -> GND
- R6 pad 1: Net-(R6-Pad1) -> LIPO_5V
- R6 pad 2: GND -> Net-(U1-FB)
- R7 pad 2: Net-(R6-Pad1) -> GND
- U4 pad 29: VTX_TX -> USART3_TX
- U4 pad 30: unconnected-(U4-PB11-Pad30) -> USART3_RX
- U4 pad 58: RECEIVER_RX -> USART1_TX
- U4 pad 59: RECEIVER_TX -> USART1_RX
Routing:
- net GND: track 0.00 -> 182.7 mm, vias 0 -> 57
- net VDD: track 0.00 -> 48.8 mm, vias 0 -> 9
- net +5V: track 0.00 -> 42.7 mm, vias 0 -> 10
- net BAT_POWER_PROTECTED: track 0.00 -> 37.3 mm
- net LIPO_5V: track 0.00 -> 33.8 mm
- net +9V: track 0.00 -> 33.5 mm
- net Net-(U10-ST): track 0.00 -> 28.5 mm, vias 0 -> 3
- net Net-(U10-~{CE}): track 0.00 -> 26.1 mm, vias 0 -> 3
- net VACC: track 0.00 -> 16.7 mm
- net BAT_CURR: track 0.00 -> 16.1 mm, vias 0 -> 1
- net Net-(U4-NRST): track 0.00 -> 14.5 mm
- net USB_D+: track 0.00 -> 13.7 mm
- net USB_D-: track 0.00 -> 13.6 mm
- net PB13: track 0.00 -> 12.9 mm, vias 0 -> 1
- net USB_5V: track 5.68 -> 16.4 mm
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- added copper zone on In2.Cu, net +5V
- added copper zone on In1.Cu, net GND
- added copper zone on In2.Cu, net VDD
- removed copper zone on In2.Cu, net GND
Other:
- board text added: "+"
- board text added: "-"
- board text added: "5V"
- board text added: "5v"
- board text added: "9V"
- board text added: "9v"
- board text added: "GND"
- board text added: "RX"
- board text added: "TX"
- board text added: "VDD"
- board text added: "buzzer"
- board text added: "camera"
- board text added: "dji vtx"
- board text added: "osd"
- board text added: "out"
- board text added: "power"
- board text added: "rx"
- board text added: "tx"
- board text added: "uart(s1)"
- board text added: "uart(s3)"
- board text added: "vidin"
- board text removed: "lilex"

Commit message: push
Parts:
- removed C48: 22pf, Capacitor_SMD:C_0402_1005Metric
- removed C50: 22uf, Capacitor_SMD:C_1206_3216Metric
- removed D5: LED, LED_SMD:LED_0603_1608Metric
- removed FB1: FerriteBead, Inductor_SMD:L_0603_1608Metric
- removed Q3: NPN, Package_TO_SOT_SMD:SOT-416
- removed R17: 10k, Resistor_SMD:R_0402_1005Metric
- removed R18: 1k, Resistor_SMD:R_0402_1005Metric
- removed U11: LM43603DSUR, easyeda2kicad:SON-16_L5.0-W4.0-P0.50-TL-EP
- removed X1: XL2EL89CSI-111YLC-27M, easyeda2kicad:CRYSTAL-SMD_4P-L3.2-W2.5-BL_SIT8008BI
- added C42: 100nf, Capacitor_SMD:C_0402_1005Metric, F.Cu at (57.3, 53.6)
- added C43: 100nf, Capacitor_SMD:C_0402_1005Metric, F.Cu at (54.0, 57.4)
- added C49: 100nf, Capacitor_SMD:C_0402_1005Metric, F.Cu at (47.4, 58.7)
- added C51: 100nf, Capacitor_SMD:C_0402_1005Metric, F.Cu at (57.3, 51.9)
- added J12: Micro_SD_Card, Connector_Card:microSD_HC_Molex_47219-2001, B.Cu at (47.5, 36.8)
- added J26: Conn_01x01, footprint_lib:signal_pad, F.Cu at (53.8, 31.6)
- added J27: Conn_01x01, footprint_lib:signal_pad, F.Cu at (56.3, 31.6)
- added J28: Conn_01x01, footprint_lib:signal_pad, F.Cu at (51.3, 31.6)
- added J29: Conn_01x01, footprint_lib:signal_pad, F.Cu at (58.8, 31.6)
- added L3: 3.3u, footprint_lib:L_pol_2016, F.Cu at (42.6, 47.3)
- added R20: 10k, Resistor_SMD:R_0402_1005Metric, F.Cu at (44.2, 37.1)
- added R25: 0, Resistor_SMD:R_0402_1005Metric, F.Cu at (33.2, 55.5)
- added R26: 1k, Resistor_SMD:R_0402_1005Metric, F.Cu at (57.8, 50.5)
- added R27: 10k, Resistor_SMD:R_0402_1005Metric, F.Cu at (50.9, 37.1)
- added R28: 10k, Resistor_SMD:R_0402_1005Metric, F.Cu at (52.0, 37.1)
- added R29: 10k, Resistor_SMD:R_0402_1005Metric, F.Cu at (55.2, 43.3)
- added R30: 10k, Resistor_SMD:R_0402_1005Metric, F.Cu at (52.5, 40.2)
- added R8: 33r, Resistor_SMD:R_0402_1005Metric, F.Cu at (42.9, 44.8)
- added U8: BMP280, Package_LGA:Bosch_LGA-8_2x2.5mm_P0.65mm_ClockwisePinNumbering, F.Cu at (54.6, 40.5)
- C10, C9: value 22pf -> 15p
- C16, C29, C38, C39, C40, C41, D4, R12, R13, R3: moved to F.Cu
- C17: value 22uf -> 100n; footprint Capacitor_SMD:C_1206_3216Metric -> Capacitor_SMD:C_0402_1005Metric; moved to F.Cu
- C18: value 22pf -> 22u; footprint Capacitor_SMD:C_0402_1005Metric -> Capacitor_SMD:C_0805_2012Metric
- C19: value 470nf -> 10u; footprint Capacitor_SMD:C_0603_1608Metric -> Capacitor_SMD:C_1210_3225Metric
- C2, C3: value 2.2uf -> 4.7u
- C20: value 2.2uF -> 22u; footprint Capacitor_SMD:C_0402_1005Metric -> Capacitor_SMD:C_0805_2012Metric
- C28, C32: value 100nf -> 1uf; moved to F.Cu
- C30: value 100nf -> 22u; footprint Capacitor_SMD:C_0402_1005Metric -> Capacitor_SMD:C_0805_2012Metric
- C31: value 22uf -> 4.7u; footprint Capacitor_SMD:C_1206_3216Metric -> Capacitor_SMD:C_0402_1005Metric; moved to F.Cu
- C33: value 22uf -> 100n; footprint Capacitor_SMD:C_0805_2012Metric -> Capacitor_SMD:C_0402_1005Metric; moved to F.Cu
- C34: value 22uf -> 10u; footprint Capacitor_SMD:C_0805_2012Metric -> Capacitor_SMD:C_1210_3225Metric
- C35: value 33pf -> 100nf; moved to F.Cu
- C36: value 33pf -> 22u; footprint Capacitor_SMD:C_0402_1005Metric -> Capacitor_SMD:C_0805_2012Metric
- C37: value 1uF -> 100nf; moved to F.Cu
- C44: value 470nf -> 10uf; footprint Capacitor_SMD:C_0603_1608Metric -> Capacitor_SMD:C_0805_2012Metric; moved to F.Cu
- C45: value 2.2uF -> 100nf; moved to F.Cu
- C46: value 22uf -> 100nf; footprint Capacitor_SMD:C_1206_3216Metric -> Capacitor_SMD:C_0402_1005Metric; moved to F.Cu
- C47: value 1uF -> 2.2uf; moved to F.Cu
- C7: value 100nf -> 4.7u
- C8: value 1uf -> 100n
- D6: footprint easyeda2kicad:SMA_L4.3-W2.6-LS5.2-RD -> Diode_SMD:D_SMA
- L1, L2: value 2.2uH -> 22uH; footprint easyeda2kicad:IND-SMD_L4.8-W4.5 -> Inductor_SMD:L_Cenker_CKCS5040
- Q1: footprint easyeda2kicad:SOT-23-3_L2.9-W1.3-P1.90-LS2.4-BR -> Package_TO_SOT_SMD:SOT-23; moved to F.Cu
- R10: value 75 -> 100k; footprint Resistor_SMD:R_0603_1608Metric -> Resistor_SMD:R_0402_1005Metric; moved to F.Cu
- R14: value 75 -> 24.9k; footprint Resistor_SMD:R_0603_1608Metric -> Resistor_SMD:R_0402_1005Metric
- R22: value 17.8k -> 10k; moved to F.Cu
- R23: value 1M -> 10k; moved to F.Cu
- R24: value 127k -> 10k; moved to F.Cu
- R5: value 249k -> 100k; moved to F.Cu
- R6: value 1M -> 24.9k; moved to F.Cu
- R7: value 17.8k -> 100k; moved to F.Cu
- R9: value 1k -> 100k
- U1: value LM43603DSUR -> MP9943GQ(TOKMAS); footprint easyeda2kicad:SON-16_L5.0-W4.0-P0.50-TL-EP -> easyeda2kicad:QFN-8_L3.0-W3.0-P0.65-BL; moved to F.Cu
- U10, U9: value LM66100DCKR -> LM66100DCK; footprint easyeda2kicad:SC-70-6_L2.0-W1.3-P0.65-LS2.1-BL -> Package_TO_SOT_SMD:SOT-363_SC-70-6; moved to F.Cu
- U2: value TLV75533PDBVR -> TLV75533PDBV; footprint easyeda2kicad:SOT-23-5_L3.0-W1.7-P0.95-LS2.8-BR -> Package_TO_SOT_SMD:SOT-23-5
- U3: value W25Q128JVSIQTR -> W25Q128JVP; footprint easyeda2kicad:SOIC-8_L5.3-W5.3-P1.27-LS8.0-BL -> Package_SON:WSON-8-1EP_6x5mm_P1.27mm_EP3.4x4.3mm
- U4: value STM32F405RGTx -> RP2350_80QFN; footprint Package_QFP:LQFP-64_10x10mm_P0.5mm -> footprint_lib:RP2350-QFN-80-1EP_10x10_P0.4mm_EP3.4x3.4mm_ThermalVias
- U5: footprint easyeda2kicad:LGA-14_L3.0-W2.5-P0.50-TL -> Package_LGA:Bosch_LGA-14_3x2.5mm_P0.5mm
- U6: value LP5907MFX-3.3/NOPB -> LP5907MFX-3.3; footprint easyeda2kicad:SOT-23-5_L3.0-W1.7-P0.95-LS2.8-BR -> Package_TO_SOT_SMD:SOT-23-5
- U7: value AT7456E -> MP9943GQ(TOKMAS); footprint easyeda2kicad:TSSOP-28_L9.7-W4.4-P0.65-LS6.4-BL-EP-2 -> easyeda2kicad:QFN-8_L3.0-W3.0-P0.65-BL; moved to F.Cu
- USB1: value TYPE-C 16PIN 2MD(073) -> USB_C_Receptacle_USB2.0_14P; footprint easyeda2kicad:USB-C-SMD_TYPE-C-6PIN-2MD-073 -> Connector_USB:USB_C_Receptacle_G-Switch_GT-USB-7010ASV
- Y1: value C115962 -> ABM8-272-T3; footprint easyeda2kicad:CRYSTAL-SMD_L5.0-W3.2 -> Crystal:Crystal_SMD_3225-4Pin_3.2x2.5mm
- moved J13 36.1 mm to (48.0, 31.6), turned to 180 degrees
- moved J5 35.3 mm to (40.3, 66.3), turned to 0 degrees
- moved J18 35.2 mm to (49.3, 66.3), turned to 0 degrees
- moved J8 34.5 mm to (45.6, 31.6), turned to 180 degrees
- moved J9 34.5 mm to (43.1, 31.6), turned to 180 degrees
- moved J15 34.4 mm to (42.6, 66.3), turned to 0 degrees
- moved J17 34.4 mm to (47.1, 66.3), turned to 0 degrees
- moved J14 34.2 mm to (40.7, 31.6), turned to 180 degrees
- moved J16 34.1 mm to (44.8, 66.3), turned to 0 degrees
- moved J23 33.8 mm to (52.2, 65.9), turned to 0 degrees
- moved J4 33.8 mm to (59.0, 65.9), turned to 0 degrees
- moved J24 33.2 mm to (54.5, 65.9), turned to 0 degrees
- moved J25 33.2 mm to (56.7, 65.9), turned to 0 degrees
- moved R1 32.9 mm to (32.2, 55.5)
- moved D3 32.0 mm to (56.0, 36.5), turned to 90 degrees
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Connections:
- C1 pad 1: GND -> VDD
- C1 pad 2: VDD -> GND
- C10 pad 1: GND -> /XIN
- C10 pad 2: Net-(U4-PH0) -> GND
- C11 pad 1: Net-(U4-NRST) -> GND
- C11 pad 2: GND -> +1V1
- C12 pad 1: GND -> VDD
- C12 pad 2: VDD -> GND
- C17 pad 1: BAT_POWER_PROTECTED -> GND
- C17 pad 2: GND -> BAT_POW_PROT
- C18 pad 1: Net-(U1-FB) -> LIPO_5V
- C18 pad 2: LIPO_5V -> GND
- C19 pad 1: Net-(U1-CBOOT) -> BAT_POW_PROT
- C19 pad 2: Net-(C19-Pad2) -> GND
- C2 pad 1: GND -> +1V1
- C2 pad 2: Net-(U4-VCAP_2) -> GND
- C20 pad 1: Net-(U1-VCC) -> LIPO_5V
- C26 pad 1: VACC -> VCC
- C28 pad 1: GND -> Net-(U1-VCC)
- C28 pad 2: VDD -> GND
- C29 pad 1: GND -> Net-(U1-BST)
- C29 pad 2: VDD -> Net-(U1-SW)
- C3 pad 1: GND -> /VREG_AVDD
- C3 pad 2: Net-(U4-VCAP_1) -> GND
- C30 pad 1: GND -> +9V
- C30 pad 2: VDD -> GND
- C31 pad 1: LIPO_5V -> +1V1
- C32 pad 1: CAM_VID_OUT -> Net-(U7-VCC)
- C32 pad 2: Net-(U7-VIN) -> GND
- C33 pad 1: Net-(U7-VOUT) -> GND
- C33 pad 2: Net-(C33-Pad2) -> BAT_POW_PROT
- C34 pad 1: Net-(U7-SAG) -> BAT_POW_PROT
- C34 pad 2: Net-(C33-Pad2) -> GND
- C35 pad 1: Net-(U7-XFB) -> Net-(U7-BST)
- C35 pad 2: GND -> Net-(U7-SW)
- C36 pad 1: Net-(U7-CLKIN) -> +9V
- C37 pad 1: LIPO_5V -> VDD
- C4 pad 1: GND -> VDD
- C4 pad 2: VDD -> GND
- C44 pad 1: Net-(U11-CBOOT) -> VDD
- C44 pad 2: Net-(C44-Pad2) -> GND
- C45 pad 1: Net-(U11-VCC) -> VDD
- C46 pad 1: +9V -> VACC
- C47 pad 1: +9V -> VACC
- C5 pad 1: GND -> VDD
- C5 pad 2: VDD -> GND
- C6 pad 1: GND -> VDD
- C6 pad 2: VDD -> GND
- C7 pad 1: Net-(U4-VDDA) -> VDD
- C8 pad 1: Net-(U4-VDDA) -> +1V1
- C9 pad 1: Net-(U4-PH1) -> Net-(C9-Pad1)
- D6 pad 1: BAT_POWER_PROTECTED -> BAT_POW_PROT
- D8 pad 1: BAT_POWER_PROTECTED -> BAT_POW_PROT
- J1 pad 1: CAM_VID_OUT -> GND
- J13 pad 1: OSD_VID_OUT -> +5V
- J14 pad 1: +5V -> GND
- J16 pad 1: DJI_RX -> DJI_RX0
- J17 pad 1: DJI_TX -> DJI_TX0
- J3 pad 1: GND -> +5V
- J6 pad 1: USART3_RX -> USART1_RX
- J7 pad 1: USART3_TX -> USART1_TX
- J8 pad 1: USART1_RX -> PIO_UART2_RX
- J9 pad 1: USART1_TX -> PIO_UART2_TX
- L1 pad 1: Net-(C19-Pad2) -> Net-(U1-SW)
- L2 pad 1: Net-(C44-Pad2) -> Net-(U7-SW)
- Q1 pad 1: PB13 -> buzz
- R1 pad 1: GND -> /~{USB_BOOT}
- R1 pad 2: Net-(U4-BOOT0) -> /QSPI_SS
- R10 pad 1: GND -> Net-(U7-VCC)
- R10 pad 2: Net-(U7-VIN) -> Net-(U7-PG)
- R14 pad 1: OSD_VID_OUT -> GND
- R14 pad 2: Net-(C33-Pad2) -> Net-(U7-FB)
- R15 pad 1: Net-(USB1-CC1) -> Net-(USB1-CC2)
- R16 pad 2: Net-(USB1-CC2) -> Net-(USB1-CC1)
- R19 pad 2: PB1 -> yellow_led
- R2 pad 1: VDD -> GND
- R2 pad 2: Net-(U4-NRST) -> Net-(R2-Pad2)
- R21 pad 2: PB0 -> green_led
- R22 pad 1: Net-(U11-RT) -> VDD
- R22 pad 2: GND -> DAT3
- R23 pad 1: +9V -> VDD
- R23 pad 2: Net-(U11-FB) -> CMD
- R24 pad 1: Net-(U11-FB) -> VDD
- R24 pad 2: GND -> SD_CLK
- R5 pad 2: GND -> LIPO_5V
- R6 pad 1: LIPO_5V -> GND
- R7 pad 1: Net-(U1-RT) -> Net-(U1-VCC)
- R7 pad 2: GND -> Net-(U1-PG)
- R9 pad 1: VDD -> Net-(U7-FB)
- R9 pad 2: Net-(U7-~{RESET}) -> +9V
- SW1 pad 1: VDD -> GND
- SW1 pad 2: Net-(U4-BOOT0) -> /~{USB_BOOT}
- SW2 pad 1: GND -> Net-(R2-Pad2)
- SW2 pad 2: Net-(U4-NRST) -> Net-(U4-RUN)
- U1 pad 1: Net-(C19-Pad2) -> Net-(U1-FB)
- U1 pad 2: Net-(C19-Pad2) -> Net-(U1-VCC)
- U1 pad 3: Net-(C19-Pad2) -> BAT_POW_PROT
- U1 pad 4: Net-(U1-CBOOT) -> Net-(U1-BST)
- U1 pad 5: Net-(U1-VCC) -> GND
- U1 pad 6: LIPO_5V -> Net-(U1-SW)
- U1 pad 7: GND -> BAT_POW_PROT
- U1 pad 8: Net-(U1-RT) -> Net-(U1-PG)
- U10 pad 5: Net-(U10-ST) -> unconnected-(U10-ST-Pad5)
- U3 pad 1: PB12 -> /QSPI_SS
- U3 pad 2: PB14 -> /QSPI_SD1
- U3 pad 3: unconnected-(U3-IO2-Pad3) -> /QSPI_SD2
- U3 pad 5: PB15 -> /QSPI_SD0
- U3 pad 6: PB13 -> /QSPI_SCLK
- U3 pad 7: unconnected-(U3-IO3-Pad7) -> /QSPI_SD3
- U4 pad 1: VDD -> USART1_TX
- U4 pad 10: LED_4 -> +1V1
- U4 pad 11: BAT_VOLTAGE -> LED_1
- U4 pad 12: GND -> LED_2
- U4 pad 13: Net-(U4-VDDA) -> LED_3
- U4 pad 14: MOTOR_1 -> LED_4
- U4 pad 15: MOTOR_2 -> VDD
- U4 pad 16: MOTOR_3 -> unconnected-(U4-GPIO16-Pad16)
- U4 pad 17: MOTOR_4 -> unconnected-(U4-GPIO17-Pad17)
- U4 pad 18: GND -> unconnected-(U4-GPIO18-Pad18)
- U4 pad 19: VDD -> unconnected-(U4-GPIO19-Pad19)
- U4 pad 2: unconnected-(U4-PC13-Pad2) -> USART1_RX
- U4 pad 20: PA4 -> buzz
- U4 pad 21: PA5 -> PIO_UART2_RX
- U4 pad 22: PA6 -> PIO_UART2_TX
- U4 pad 23: PA7 -> unconnected-(U4-GPIO23-Pad23)
- U4 pad 24: BAT_CURR -> VDD
- U4 pad 26: PB0 -> unconnected-(U4-GPIO25-Pad26)
- U4 pad 27: PB1 -> unconnected-(U4-GPIO26-Pad27)
- U4 pad 28: LED_1 -> IMU_INT
- U4 pad 29: USART3_TX -> VDD
- U4 pad 3: unconnected-(U4-PC14-Pad3) -> MOTOR_1
- U4 pad 30: USART3_RX -> /XIN
- U4 pad 31: Net-(U4-VCAP_1) -> /XOUT
- U4 pad 32: VDD -> +1V1
- U4 pad 33: PB12 -> /SWCLK
- U4 pad 34: PB13 -> /SWD
- U4 pad 35: PB14 -> Net-(U4-RUN)
- U4 pad 36: PB15 -> IMU_SDO
- U4 pad 37: DJI_RX -> IMU_CS
- U4 pad 38: DJI_TX -> IMU_CLK
- U4 pad 39: unconnected-(U4-PC8-Pad39) -> IMU_SDA
- U4 pad 4: unconnected-(U4-PC15-Pad4) -> MOTOR_2
- U4 pad 40: OSD_CS -> I2C_SDA
- U4 pad 41: PA8 -> VDD
- U4 pad 42: unconnected-(U4-PA9-Pad42) -> I2C_SCK
- U4 pad 43: unconnected-(U4-PA10-Pad43) -> SD_CLK
- U4 pad 44: USB_D- -> CMD
- U4 pad 45: USB_D+ -> DAT0
- U4 pad 46: unconnected-(U4-PA13-Pad46) -> DAT1
- U4 pad 47: Net-(U4-VCAP_2) -> DAT2
- U4 pad 48: VDD -> DAT3
- U4 pad 5: Net-(U4-PH0) -> VDD
- U4 pad 50: unconnected-(U4-PA15-Pad50) -> VDD
- U4 pad 51: OSD_CLK -> +1V1
- U4 pad 52: OSD_SDOUT -> BAT_CURR
- U4 pad 53: OSD_SDIN -> TELEMETRY
- U4 pad 54: TELEMETRY -> unconnected-(U4-GPIO43_ADC3-Pad54)
- U4 pad 55: unconnected-(U4-PB3-Pad55) -> BAT_VOLTAGE
- U4 pad 56: unconnected-(U4-PB4-Pad56) -> green_led
- U4 pad 57: LED_2 -> yellow_led
- U4 pad 58: USART1_TX -> unconnected-(U4-GPIO47_ADC7-Pad58)
- U4 pad 59: USART1_RX -> VDD
- U4 pad 6: Net-(U4-PH1) -> MOTOR_3
- U4 pad 60: Net-(U4-BOOT0) -> VDD
- U4 pad 61: unconnected-(U4-PB8-Pad61) -> /VREG_AVDD
- U4 pad 62: unconnected-(U4-PB9-Pad62) -> GND
- U4 pad 63: GND -> /VREG_LX
- U4 pad 7: Net-(U4-NRST) -> MOTOR_4
- U4 pad 9: LED_3 -> unconnected-(U4-GPIO11-Pad9)
- U5 pad 1: PA6 -> IMU_SDO
- U5 pad 12: PA8 -> IMU_CS
- U5 pad 13: PA5 -> IMU_CLK
- U5 pad 14: PA7 -> IMU_SDA
- U5 pad 4: unconnected-(U5-INT1/INT-Pad4) -> IMU_INT
- U5 pad 5: VACC -> VCC
- U7 pad 1: unconnected-(U7-NC-Pad1) -> Net-(U7-FB)
- U7 pad 2: unconnected-(U7-NC-Pad2) -> Net-(U7-VCC)
- U7 pad 3: VDD -> BAT_POW_PROT
- U7 pad 4: GND -> Net-(U7-BST)
- U7 pad 5: Net-(U7-CLKIN) -> GND
- U7 pad 6: Net-(U7-XFB) -> Net-(U7-SW)
- U7 pad 7: unconnected-(U7-CLKOUT-Pad7) -> BAT_POW_PROT
- U7 pad 8: OSD_CS -> Net-(U7-PG)
- Y1 pad 1: Net-(U4-PH0) -> /XIN
- Y1 pad 2: Net-(U4-PH1) -> GND
Routing:
- net GND: track 182.7 -> 1.07 mm, vias 57 -> 4
- net BAT_POWER_PROTECTED: track 37.3 -> 0.00 mm
- net +9V: track 33.5 -> 0.00 mm
- net I2C1_SDA: track 0.00 -> 31.7 mm, vias 0 -> 2
- net I2C1_SCL: track 0.00 -> 29.4 mm, vias 0 -> 2
- net Net-(U10-ST): track 28.5 -> 0.00 mm, vias 3 -> 0
- net +5V: track 42.7 -> 17.5 mm, vias 10 -> 3
- net MOTOR_2: track 0.00 -> 24.6 mm, vias 0 -> 2
- net MOTOR_1: track 0.00 -> 24.4 mm, vias 0 -> 2
- net Net-(U10-~{CE}): track 26.1 -> 3.29 mm, vias 3 -> 0
- net MOTOR_4: track 0.00 -> 22.6 mm, vias 0 -> 2
- net MOTOR_3: track 0.00 -> 22.5 mm, vias 0 -> 2
- net TELEMETRY: track 0.00 -> 18.9 mm, vias 0 -> 2
- net BAT_VOLTAGE: track 1.70 -> 18.7 mm, vias 0 -> 2
- net VACC: track 16.7 -> 0.00 mm
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- added copper zone on B.Cu, net GND
- added copper zone on F.Cu, net GND
- added copper zone on In2.Cu, net GND
- removed copper zone on In2.Cu, net +5V
- removed copper zone on In2.Cu, net VDD
Other:
- board text added: "I2C"
- board text added: "dji"
- board text added: "scl"
- board text added: "sda"
- board text added: "uart1"
- board text added: "uart2"
- board text removed: "5v"
- board text removed: "camera"
- board text removed: "dji vtx"
- board text removed: "osd"
- board text removed: "out"
- board text removed: "uart(s1)"
- board text removed: "uart(s3)"
- board text removed: "vidin"

Commit message: finished routinnnn
:3
Parts:
- added C48: 10uf, Capacitor_SMD:C_0805_2012Metric, F.Cu at (58.6, 54.8)
- moved D1 2.27 mm to (56.0, 36.5)
- moved D3 2.27 mm to (58.3, 36.5)
- moved C36 1.16 mm to (54.1, 55.6)
- moved Q1 0.53 mm to (39.3, 59.5)
- moved C17 0.52 mm to (61.7, 59.6)
- moved R11 0.39 mm to (40.0, 39.7)
- moved C42 0.32 mm to (57.3, 53.3)
- moved C41 0.30 mm to (41.5, 38.6)
- moved C11 0.28 mm to (50.4, 43.2)
- moved C21 0.28 mm to (49.5, 43.2)
- moved C6 0.27 mm to (51.4, 43.2)
- moved R3 0.18 mm to (55.6, 60.3)
- moved D6 0.14 mm to (66.1, 41.0)
- moved D8 0.14 mm to (60.9, 43.0)
- moved R30 0.14 mm to (52.5, 40.4)
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Routing:
- net +5V: track 17.5 -> 159.4 mm, vias 3 -> 8
- net VDD: track 39.6 -> 173.1 mm, vias 1 -> 10
- net +9V: track 0.00 -> 71.5 mm, vias 0 -> 2
- net LED_1: track 4.19 -> 62.6 mm, vias 1 -> 2
- net PIO_UART2_TX: track 0.00 -> 53.5 mm, vias 0 -> 2
- net PIO_UART2_RX: track 0.00 -> 51.8 mm, vias 0 -> 2
- net LED_4: track 2.59 -> 54.3 mm, vias 1 -> 4
- net /~{USB_BOOT}: track 0.00 -> 51.0 mm
- net +1V1: track 14.9 -> 59.6 mm, vias 0 -> 5
- net LED_2: track 3.12 -> 46.7 mm, vias 1 -> 2
- net Net-(U10-~{CE}): track 3.29 -> 46.7 mm, vias 0 -> 2
- net BAT_POW_PROT: track 8.21 -> 44.8 mm, vias 0 -> 3
- net VACC: track 0.00 -> 22.1 mm, vias 0 -> 2
- net LED_3: track 2.66 -> 22.5 mm, vias 1 -> 3
- net buzz: track 0.90 -> 17.4 mm, vias 1 -> 2
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
Commit message: a
Other:
- outline, holes or cut-outs redrawn

Commit message: a
Parts:
- added J30: Conn_01x01, TestPoint:TestPoint_Pad_1.0x1.0mm, F.Cu at (68.5, 61.6)
- added J31: Conn_01x01, TestPoint:TestPoint_Pad_1.0x1.0mm, F.Cu at (62.5, 30.2)
- added J32: Conn_01x01, TestPoint:TestPoint_Pad_1.0x1.0mm, F.Cu at (31.1, 36.4)
- moved J19 40.3 mm to (35.4, 63.2), turned to 180 degrees
- moved J21 40.3 mm to (64.1, 34.9), turned to 0 degrees
- moved J20 40.1 mm to (63.9, 63.1), turned to -90 degrees
- moved J22 40.1 mm to (35.7, 34.7), turned to 90 degrees
- moved D8 2.11 mm to (60.8, 45.2)
- moved C25 0.78 mm to (60.9, 45.8)
- moved C27 0.78 mm to (61.8, 45.8)
Connections:
- U4 pad 11: LED_1 -> unconnected-(U4-GPIO12-Pad11)
- U4 pad 12: LED_2 -> unconnected-(U4-GPIO13-Pad12)
- U4 pad 13: LED_3 -> LED_1
- U4 pad 14: LED_4 -> unconnected-(U4-GPIO15-Pad14)
- U4 pad 27: unconnected-(U4-GPIO26-Pad27) -> IMU_CLKIN
- U5 pad 9: GND -> IMU_CLKIN
Routing:
- net LED_1: track 62.6 -> 22.1 mm, vias 2 -> 3
- net LED_4: track 54.3 -> 31.2 mm, vias 4 -> 0
- net LED_2: track 46.7 -> 31.4 mm
- net IMU_CLKIN: track 0.00 -> 12.8 mm, vias 0 -> 2
- net LED_3: track 22.5 -> 31.6 mm, vias 3 -> 2
- net BAT_POW_PROT: track 44.8 -> 47.0 mm
