File: src/hardware/fc/drone.kicad_sch (KiCad schematic)
At the start: 117 parts, among them J1 Conn_01x01, J10 Conn_01x01, J11 Conn_01x01, J12 Conn_01x01, J13 Conn_01x01, J14 Conn_01x01, J15 Conn_01x01, J16 Conn_01x01, J17 Conn_01x01, J18 Conn_01x01, J19 Conn_01x03, J2 Conn_01x08, J20 Conn_01x03, J21 Conn_01x03, J22 Conn_01x03, J23 Conn_01x01, J24 Conn_01x01, J25 Conn_01x01, J3 Conn_01x01, J4 Conn_01x01, J5 Conn_01x01, J6 Conn_01x01, J7 Conn_01x01, J8 Conn_01x01, J9 Conn_01x01, Q1 AO3400A, Q2 NPN, Q3 NPN, SW1 SW_Push, SW2 SW_Push, U10 LM66100DCKR, U2 TLV75533PDBVR, U3 W25Q128JVSIQTR, U4 STM32F405RGTx, U5 ICM-42688-P, U6 LP5907MFX-3.3/NOPB, U7 AT7456E, U8 MP4420HGJ-Z, U9 LM66100DCKR, X1 XL2EL89CSI-111YLC-27M, Y1 C115962

Commit message: pcb update
Parts:
- removed C42, C43: 22uf, Capacitor_SMD:C_1206_3216Metric, symbol Device:C
- removed J12: Conn_01x01, footprint_lib:signal_pad, symbol Connector_Generic:Conn_01x01
- removed R20: 150k, Resistor_SMD:R_0603_1608Metric, symbol Device:R
- removed R8: 41.2k, Resistor_SMD:R_0402_1005Metric, symbol Device:R
- removed U8: MP4420HGJ-Z, easyeda2kicad:TSOT-23-8_L2.9-W1.6-P0.65-LS2.8-BL, symbol easyeda2kicad:MP4420HGJ-Z
- added C44: 470nf, Capacitor_SMD:C_0603_1608Metric, symbol Device:C
- added C45: 2.2uF, Capacitor_SMD:C_0402_1005Metric, symbol Device:C
- added C46, C50: 22uf, Capacitor_SMD:C_1206_3216Metric, symbol Device:C
- added C47: 1uF, Capacitor_SMD:C_0402_1005Metric, symbol Device:C
- added C48: 22pf, Capacitor_SMD:C_0402_1005Metric, symbol Device:C
- added L2: 2.2uH, easyeda2kicad:IND-SMD_L4.8-W4.5, symbol Device:L
- added R22: 17.8k, Resistor_SMD:R_0402_1005Metric, symbol Device:R
- added R23: 1M, Resistor_SMD:R_0402_1005Metric, symbol Device:R
- added R24: 127k, Resistor_SMD:R_0402_1005Metric, symbol Device:R
- added U1, U11: LM43603DSUR, easyeda2kicad:SON-16_L5.0-W4.0-P0.50-TL-EP, symbol easyeda2kicad:LM43603DSUR
- C17: value 100nf -> 22uf; footprint Capacitor_SMD:C_0402_1005Metric -> Capacitor_SMD:C_1206_3216Metric; LCSC Part C1525 -> C342620
- C18: value 100nf -> 22pf; LCSC Part C1525 -> C1555
- C19: value 22uf -> 470nf; footprint Capacitor_SMD:C_0805_2012Metric -> Capacitor_SMD:C_0603_1608Metric; LCSC Part C45783 -> C1623
- C20: value 100nf -> 2.2uF; LCSC Part C1525 -> C60078
- C37: value 22uf -> 1uF; footprint Capacitor_SMD:C_0805_2012Metric -> Capacitor_SMD:C_0402_1005Metric; LCSC Part C45783 -> C52923
- L1: value 1OuH -> 2.2uH; footprint Inductor_SMD:L_KOHERelec_MDA7030 -> easyeda2kicad:IND-SMD_L4.8-W4.5; LCSC Part C2847485 -> C133191
- R5: value 20 -> 249k; LCSC Part C25089 -> C11425
- R6: value 7.68k -> 1M; LCSC Part C25919 -> C26083
- R7: value 51k -> 17.8k; LCSC Part C25794 -> C77605
Connections:
- net +5V: no longer J7.1 (Pin_1)
- net +9V: now also C46.1, C47.1, C48.2, L2.2, R23.1, U11.6 (BIAS)
- net GND: now also C17.2, C31.2, C37.2, R5.2, R7.2, C45.2, C46.2, C47.2, C50.2, R22.2, R24.2, U1.15 (PGND), U1.16 (PGND), U1.17 (EP), U1.7 (SYNC), U11.15 (PGND), U11.16 (PGND), U11.17 (EP), U11.7 (SYNC); no longer C17.1, C19.1, C31.1, C37.1, J6.1 (Pin_1), R6.2
- net LIPO_5V: now also C18.2, C31.1, C37.1, R6.1, U1.6 (BIAS); no longer C19.2, C37.2
- net BAT_POWER_PROTECTED: now reaches D6.1 (K), D8.1 (A1)
- net BAT_POWER_PROTECTED: now also C17.1, C50.1, U1.12 (EN), U1.13 (VIN), U1.14 (VIN), U11.12 (EN), U11.13 (VIN), U11.14 (VIN); no longer C20.1, C31.2
- net at C18.1: now also R5.1, R6.2, U1.10 (FB); no longer L1.1
- net at R7.1: now also U1.8 (RT)
- net USART3_RX: now reaches U4.30 (PB11)
- net USART3_RX: now also J6.1 (Pin_1)
- net RECEIVER_RX renamed USART1_RX
- net USART1_RX: now also U4.59 (PB7); no longer U4.58 (PB6)
- net RECEIVER_TX renamed USART1_TX
- net USART1_TX: now also U4.58 (PB6); no longer U4.59 (PB7)
- net VTX_TX renamed USART3_TX
- net USART3_TX: now also J7.1 (Pin_1)
- new net: R22.1, U11.8 (RT)
- new net: C48.1, R23.2, R24.1, U11.10 (FB)
- new net: C20.1, U1.5 (VCC)
- new net: C44.1, U11.4 (CBOOT)
- new net: C44.2, L2.1, U11.1 (SW), U11.2 (SW), U11.3 (SW)
- new net: C19.1, U1.4 (CBOOT)
- new net: C19.2, L1.1, U1.1 (SW), U1.2 (SW), U1.3 (SW)
- new net: C45.1, U11.5 (VCC)
Other:
- note added: "idk atp"
- note added: "uart"
- note added: "vbat to 9v (dji o3 maybe other stuff??)"
- note removed: "no components under it"
- note removed: "radiomaster rp1 nano elrs connector"
- moved on the sheet: D6, D8, J19, J20, J21, J22, J23, J24, J25

Commit message: push
Parts:
- removed C48: 22pf, Capacitor_SMD:C_0402_1005Metric, symbol Device:C
- removed C50: 22uf, Capacitor_SMD:C_1206_3216Metric, symbol Device:C
- removed D5: LED, LED_SMD:LED_0603_1608Metric, symbol Device:LED
- removed FB1: FerriteBead, Inductor_SMD:L_0603_1608Metric, symbol Device:FerriteBead
- removed Q1: AO3400A, easyeda2kicad:SOT-23-3_L2.9-W1.3-P1.90-LS2.4-BR, symbol easyeda2kicad:AO3400A
- removed Q3: NPN, Package_TO_SOT_SMD:SOT-416, symbol Simulation_SPICE:NPN
- removed R17: 10k, Resistor_SMD:R_0402_1005Metric, symbol Device:R
- removed R18: 1k, Resistor_SMD:R_0402_1005Metric, symbol Device:R
- removed U1, U11: LM43603DSUR, easyeda2kicad:SON-16_L5.0-W4.0-P0.50-TL-EP, symbol easyeda2kicad:LM43603DSUR
- removed U10, U9: LM66100DCKR, easyeda2kicad:SC-70-6_L2.0-W1.3-P0.65-LS2.1-BL, symbol easyeda2kicad:LM66100DCKR
- removed U2: TLV75533PDBVR, easyeda2kicad:SOT-23-5_L3.0-W1.7-P0.95-LS2.8-BR, symbol easyeda2kicad:TLV75533PDBVR
- removed U3: W25Q128JVSIQTR, easyeda2kicad:SOIC-8_L5.3-W5.3-P1.27-LS8.0-BL, symbol easyeda2kicad:W25Q128JVSIQTR
- removed U4: STM32F405RGTx, Package_QFP:LQFP-64_10x10mm_P0.5mm, symbol MCU_ST_STM32F4:STM32F405RGTx
- removed U6: LP5907MFX-3.3/NOPB, easyeda2kicad:SOT-23-5_L3.0-W1.7-P0.95-LS2.8-BR, symbol easyeda2kicad:LP5907MFX-3.3_NOPB
- removed U7: AT7456E, easyeda2kicad:TSSOP-28_L9.7-W4.4-P0.65-LS6.4-BL-EP-2, symbol easyeda2kicad:AT7456E
- removed USB1: TYPE-C 16PIN 2MD(073), easyeda2kicad:USB-C-SMD_TYPE-C-6PIN-2MD-073, symbol easyeda2kicad:TYPE-C16PIN2MD(073)
- removed X1: XL2EL89CSI-111YLC-27M, easyeda2kicad:CRYSTAL-SMD_4P-L3.2-W2.5-BL_SIT8008BI, symbol easyeda2kicad:XL2EL89CSI-111YLC-27M
- removed Y1: C115962, easyeda2kicad:CRYSTAL-SMD_L5.0-W3.2, symbol Device:Crystal
- added C42, C43, C49, C51: 100nf, Capacitor_SMD:C_0402_1005Metric, symbol Device:C
- added J12: Micro_SD_Card, Connector_Card:microSD_HC_Molex_47219-2001, symbol Connector:Micro_SD_Card
- added J26, J27, J28, J29: Conn_01x01, footprint_lib:signal_pad, symbol Connector_Generic:Conn_01x01
- added L3: 3.3u, footprint_lib:L_pol_2016, symbol Device:L
- added Q1: AO3400A, Package_TO_SOT_SMD:SOT-23, symbol Transistor_FET:AO3400A
- added R20, R27, R28, R29, R30: 10k, Resistor_SMD:R_0402_1005Metric, symbol Device:R
- added R25: 0, Resistor_SMD:R_0402_1005Metric, symbol Device:R
- added R26: 1k, Resistor_SMD:R_0402_1005Metric, symbol Device:R
- added R8: 33r, Resistor_SMD:R_0402_1005Metric, symbol Device:R
- added U1, U7: MP9943GQ(TOKMAS), easyeda2kicad:QFN-8_L3.0-W3.0-P0.65-BL, symbol easyeda2kicad:MP9943GQ(TOKMAS)
- added U10, U9: LM66100DCK, Package_TO_SOT_SMD:SOT-363_SC-70-6, symbol Power_Management:LM66100DCK
- added U2: TLV75533PDBV, Package_TO_SOT_SMD:SOT-23-5, symbol Regulator_Linear:TLV75533PDBV
- added U3: W25Q128JVP, Package_SON:WSON-8-1EP_6x5mm_P1.27mm_EP3.4x4.3mm, symbol Memory_Flash:W25Q128JVP
- added U4: RP2350_80QFN, footprint_lib:RP2350-QFN-80-1EP_10x10_P0.4mm_EP3.4x3.4mm_ThermalVias, symbol MCU_RaspberryPi_RP2350:RP2350_80QFN
- added U6: LP5907MFX-3.3, Package_TO_SOT_SMD:SOT-23-5, symbol Regulator_Linear:LP5907MFX-3.3
- added U8: BMP280, Package_LGA:Bosch_LGA-8_2x2.5mm_P0.65mm_ClockwisePinNumbering, symbol Sensor_Pressure:BMP280
- added USB1: USB_C_Receptacle_USB2.0_14P, Connector_USB:USB_C_Receptacle_G-Switch_GT-USB-7010ASV, symbol Connector:USB_C_Receptacle_USB2.0_14P
- added Y1: ABM8-272-T3, Crystal:Crystal_SMD_3225-4Pin_3.2x2.5mm, symbol Device:Crystal_GND24
- C10, C9: value 22pf -> 15p; LCSC Part C466226 -> (none)
- C17: value 22uf -> 100n; footprint Capacitor_SMD:C_1206_3216Metric -> Capacitor_SMD:C_0402_1005Metric; LCSC (none) -> C15195; LCSC Part C342620 -> (none)
- C18: value 22pf -> 22u; footprint Capacitor_SMD:C_0402_1005Metric -> Capacitor_SMD:C_0805_2012Metric; LCSC (none) -> C13585; LCSC Part C1555 -> (none)
- C19: value 470nf -> 10u; footprint Capacitor_SMD:C_0603_1608Metric -> Capacitor_SMD:C_1210_3225Metric; LCSC (none) -> C13585; LCSC Part C1623 -> (none)
- C2, C3: value 2.2uf -> 4.7u; LCSC Part C12530 -> (none)
- C20: value 2.2uF -> 22u; footprint Capacitor_SMD:C_0402_1005Metric -> Capacitor_SMD:C_0805_2012Metric; LCSC (none) -> C13585; LCSC Part C60078 -> (none)
- C28, C32: value 100nf -> 1uf; LCSC Part C1525 -> C52923
- C30: value 100nf -> 22u; footprint Capacitor_SMD:C_0402_1005Metric -> Capacitor_SMD:C_0805_2012Metric; LCSC (none) -> C13585; LCSC Part C1525 -> (none)
- C31: value 22uf -> 4.7u; footprint Capacitor_SMD:C_1206_3216Metric -> Capacitor_SMD:C_0402_1005Metric; LCSC Part C342620 -> (none)
- C33: value 22uf -> 100n; footprint Capacitor_SMD:C_0805_2012Metric -> Capacitor_SMD:C_0402_1005Metric; LCSC (none) -> C15195; LCSC Part C45783 -> (none)
- C34: value 22uf -> 10u; footprint Capacitor_SMD:C_0805_2012Metric -> Capacitor_SMD:C_1210_3225Metric; LCSC (none) -> C13585; LCSC Part C45783 -> (none)
- C35: value 33pf -> 100nf; LCSC Part C115628 -> C1525
- C36: value 33pf -> 22u; footprint Capacitor_SMD:C_0402_1005Metric -> Capacitor_SMD:C_0805_2012Metric; LCSC (none) -> C13585; LCSC Part C115628 -> (none)
- C37: value 1uF -> 100nf; LCSC Part C52923 -> C1525
- C44: value 470nf -> 10uf; footprint Capacitor_SMD:C_0603_1608Metric -> Capacitor_SMD:C_0805_2012Metric; LCSC Part C1623 -> C91185
- C45: value 2.2uF -> 100nf; LCSC Part C60078 -> C1525
- C46: value 22uf -> 100nf; footprint Capacitor_SMD:C_1206_3216Metric -> Capacitor_SMD:C_0402_1005Metric; LCSC Part C342620 -> C1525
- C47: value 1uF -> 2.2uf; LCSC Part C52923 -> C12530
- C7: value 100nf -> 4.7u; LCSC Part C1525 -> (none)
- C8: value 1uf -> 100n; LCSC Part C52923 -> (none)
- D6: footprint easyeda2kicad:SMA_L4.3-W2.6-LS5.2-RD -> Diode_SMD:D_SMA
- L1: value 2.2uH -> 22uH; footprint easyeda2kicad:IND-SMD_L4.8-W4.5 -> Inductor_SMD:L_Cenker_CKCS5040; LCSC Part C133191 -> (none)
- L2: value 2.2uH -> 22uH; footprint easyeda2kicad:IND-SMD_L4.8-W4.5 -> Inductor_SMD:L_Cenker_CKCS5040; LCSC Part C133191 -> C2879700
- R10: value 75 -> 100k; footprint Resistor_SMD:R_0603_1608Metric -> Resistor_SMD:R_0402_1005Metric; LCSC Part C4275 -> (none)
- R14: value 75 -> 24.9k; footprint Resistor_SMD:R_0603_1608Metric -> Resistor_SMD:R_0402_1005Metric; LCSC Part C4275 -> (none)
- R22: value 17.8k -> 10k; LCSC Part C77605 -> C25744
- R23: value 1M -> 10k; LCSC Part C26083 -> C25744
- R24: value 127k -> 10k; LCSC Part C11688 -> C25744
- R5: value 249k -> 100k; LCSC Part C11425 -> (none)
- R6: value 1M -> 24.9k; LCSC Part C26083 -> (none)
- R7: value 17.8k -> 100k; LCSC Part C77605 -> (none)
- R9: value 1k -> 100k; LCSC Part C11702 -> (none)
- U5: footprint easyeda2kicad:LGA-14_L3.0-W2.5-P0.50-TL -> Package_LGA:Bosch_LGA-14_3x2.5mm_P0.5mm
Connections:
- net USART3_RX is gone; now on net USART1_RX: J6.1 (Pin_1)
- net USART3_TX is gone; now on net USART1_TX: J7.1 (Pin_1)
- net +5V: now also J13.1 (Pin_1), J3.1 (Pin_1), J29.1 (Pin_1), U10.6 (VOUT), U2.1 (IN), U2.3 (EN), U6.1 (IN), U6.3 (EN), U9.6 (VOUT); no longer J14.1 (Pin_1)
- net +9V: now also C30.1, C36.1, R9.2; no longer C46.1, C47.1, R23.1
- net BAT_CURR: now also U4.52 (GPIO41_ADC1)
- net BAT_VOLTAGE: now also U4.55 (GPIO44_ADC4)
- net GND: now also C1.2, C10.2, C11.1, C12.2, C17.1, C18.2, C19.2, C2.2, C28.2, C3.2, C30.2, C32.2, C33.1, C34.2, C4.2, C44.2, C5.2, C6.2, J1.1 (Pin_1), J14.1 (Pin_1), R14.1, R2.1, R6.1, SW1.1, C42.2, C43.2, C49.2, C51.2, J12.6 (VSS), J12.9 (SHIELD), J28.1 (Pin_1), Q1.2 (S), U1.5 (GND), U10.2 (GND), U2.2 (GND), U3.4 (GND), U3.9 (EP), U4.62 (VREG_PGND), U4.81 (GND), U6.2 (GND), U7.5 (GND), U8.1 (GND), U8.5 (SDO), U8.7 (GND), U9.2 (GND), U9.3 (~{CE}), USB1.A1 (GND), USB1.A12 (GND), USB1.B1 (GND), USB1.B12 (GND), USB1.S1 (SHIELD), Y1.2, Y1.4; no longer C1.1, C10.1, C11.2, C12.1, C17.2, C2.1, C28.1, C29.1, C3.1, C30.1, C35.2, C4.1, C5.1, C6.1, J3.1 (Pin_1), R1.1, R10.1, R22.2, R24.2, R5.2, R7.2, SW2.1
- net LED_1: now also U4.11 (GPIO12)
- net LED_2: now also U4.12 (GPIO13)
- net LED_3: now also U4.13 (GPIO14)
- net LED_4: now also U4.14 (GPIO15)
- net LIPO_5V: now also C18.1, C20.1, R5.2, U10.1 (VIN); no longer C18.2, C31.1, C37.1, R6.1
- net MOTOR_1: now also U4.3 (GPIO6)
- net MOTOR_2: now also U4.4 (GPIO7)
- net MOTOR_3: now also U4.6 (GPIO8)
- net MOTOR_4: now also U4.7 (GPIO9)
- net TELEMETRY: now also U4.53 (GPIO42_ADC2)
- net USART1_RX: now also U4.2 (GPIO5); no longer J8.1 (Pin_1)
- net USART1_TX: now also U4.1 (GPIO4); no longer J9.1 (Pin_1)
- net USB_5V: now also U9.1 (VIN), USB1.A4 (VBUS), USB1.A9 (VBUS), USB1.B4 (VBUS), USB1.B9 (VBUS)
- net USB_D+: now also U4.67 (USB_DP), USB1.A6 (D+), USB1.B6 (D+)
- net USB_D-: now also U4.66 (USB_DM), USB1.A7 (D-), USB1.B7 (D-)
- net VACC: now also C46.1, C47.1, U6.5 (OUT), U8.8 (VDD); no longer C26.1, U5.5 (VDDIO)
- net VDD: now also C1.1, C12.1, C37.1, C4.1, C44.1, C45.1, C5.1, C6.1, C7.1, R22.1, R23.1, R24.1, C42.1, C43.1, C49.1, C51.1, J12.4 (VDD), R20.1, R25.1, R27.1, R28.1, R29.2, R30.2, R8.1, U2.5 (OUT), U3.8 (VCC), U4.15 (IOVDD), U4.24 (IOVDD), U4.29 (IOVDD), U4.41 (IOVDD), U4.5 (IOVDD), U4.50 (IOVDD), U4.59 (ADC_AVDD), U4.60 (IOVDD), U4.64 (VREG_VIN), U4.68 (USB_OTP_VDD), U4.69 (QSPI_IOVDD), U4.76 (IOVDD), U8.2 (CSB), U8.6 (VDDIO); no longer C1.2, C12.2, C28.2, C29.2, C30.2, C4.2, C5.2, C6.2, R2.1, R9.1, SW1.1
- net +1V1: now reaches C8.1
- net +1V1: now also C11.2, C2.1, C31.1, L3.1, U4.10 (DVDD), U4.32 (DVDD), U4.51 (DVDD), U4.65 (VREG_FB); no longer C7.1
- net at D4.2 (A), TP2.1: now also Q1.3 (D)
- net CMD: now reaches R23.2
- net CMD: now also J12.3 (CMD), U4.44 (GPIO35); no longer R24.1
- net at R3.1, R4.1: now also U10.3 (~{CE}), U9.5 (ST)
- net at C35.1: now also U7.4 (BST)
- net QSPI_SS: now reaches R1.2
- net QSPI_SS: now also R25.2, U3.1 (~{CS}), U4.75 (QSPI_SS); no longer SW1.2
- net at R5.1, R6.2: now also U1.1 (FB); no longer C18.1
- net IMU_INT: now reaches U5.4 (INT1/INT)
- net IMU_INT: now also U4.28 (GPIO27)
- net at L2.1: now also C35.2, U7.6 (SW); no longer C44.2
- net at R10.2: now also U7.8 (PG); no longer C32.2
- net at R15.1: now also USB1.B5 (CC2)
- net at R16.2: now also USB1.A5 (CC1)
- net BAT_POW_PROT: now reaches C34.1
- net BAT_POW_PROT: now also C17.2, C19.1, C33.2, D6.1 (K), D8.1 (A1), U1.3 (EN), U1.7 (VIN), U7.3 (EN), U7.7 (VIN)
- net at L1.1: now also C29.2, U1.6 (SW); no longer C19.2
- net at C9.1: now also R26.2, Y1.3
- net at R7.1: now also C28.1, U1.2 (VCC)
- removed net BAT_POWER_PROTECTED: C17.1, D6.1 (K), D8.1 (A1)
- net CAM_VID_OUT: no longer names the net of C32.1
- net CAM_VID_OUT: now also R10.1, U7.2 (VCC); no longer J1.1 (Pin_1)
- net DJI_RX renamed DJI_RX0
- net DJI_RX0: now also U4.77 (GPIO0)
- net DJI_TX renamed DJI_TX0
- net DJI_TX0: now also U4.78 (GPIO1)
- removed net OSD_VID_OUT: J13.1 (Pin_1), R14.1
- net PA5 renamed IMU_CLK
- net IMU_CLK: now also U4.38 (GPIO30)
- net PA6 renamed IMU_SDO
- net IMU_SDO: now also U4.36 (GPIO28)
- net PA7 renamed IMU_SDA
- net IMU_SDA: now also U4.39 (GPIO31)
- net PA8 renamed IMU_CS
- net IMU_CS: now also U4.37 (GPIO29)
- net PB0 renamed green_led
- net green_led: now also U4.56 (GPIO45_ADC5)
- net PB1 renamed yellow_led
- net yellow_led: now also U4.57 (GPIO46_ADC6)
- new net: C29.1, U1.4 (BST)
- new net: R7.2, U1.8 (PG)
- new net: R14.2, R9.1, U7.1 (FB)
- new net: R2.2, SW2.1
- new net: SW2.2, U4.35 (RUN)
- new net DAT0: J12.7 (DAT0), R27.2, U4.45 (GPIO36)
- new net DAT1: J12.8 (DAT1), R28.2, U4.46 (GPIO37)
- new net DAT2: J12.1 (DAT2), R20.2, U4.47 (GPIO38)
- new net DAT3: J12.2 (DAT3/CD), R22.2, U4.48 (GPIO39)
- new net I2C1_SCL: J27.1 (Pin_1), U4.80 (GPIO3)
- new net I2C1_SDA: J26.1 (Pin_1), U4.79 (GPIO2)
- new net I2C_SCK: R30.1, U4.42 (GPIO33), U8.4 (SCK)
- new net I2C_SDA: R29.1, U4.40 (GPIO32), U8.3 (SDI)
- new net PIO_UART2_RX: J8.1 (Pin_1), U4.21 (GPIO21)
- new net PIO_UART2_TX: J9.1 (Pin_1), U4.22 (GPIO22)
- new net QSPI_SCLK: U3.6 (CLK), U4.71 (QSPI_SCLK)
- new net QSPI_SD0: U3.5 (DI/IO_{0}), U4.72 (QSPI_SD0)
- new net QSPI_SD1: U3.2 (DO/IO_{1}), U4.74 (QSPI_SD1)
- new net QSPI_SD2: U3.3 (~{WP}/IO_{2}), U4.73 (QSPI_SD2)
- new net QSPI_SD3: U3.7 (~{HOLD}/~{RESET}/IO_{3}), U4.70 (QSPI_SD3)
- new net SD_CLK: J12.5 (CLK), R24.2, U4.43 (GPIO34)
- new net SWCLK: U4.33 (SWCLK)
- new net SWD: U4.34 (SWD)
- new net VCC: C26.1, U5.5 (VDDIO)
- new net VREG_AVDD: C3.1, R8.2, U4.61 (VREG_AVDD)
- new net VREG_LX: L3.2, U4.63 (VREG_LX)
- new net XIN: C10.1, U4.30 (XIN), Y1.1
- new net XOUT: R26.1, U4.31 (XOUT)
- new net buzz: Q1.1 (G), U4.20 (GPIO20)
- new net ~{USB_BOOT}: R1.1, SW1.2
- no-connect marks 0 -> 2
Other:
- note added: "."
- note added: "12MHz Crystal"
- note added: "baro"
- note added: "blackbox microsd card slot"
- note added: "transient and reverse polarity protection"
- note added: "vbat-9v"
- note removed: "C31 is x7r + min 35v rated C19 is ceramic"
- note removed: "JST?"
- note removed: "analog video"
- note removed: "blackbox flash chip"
- note removed: "connector"
- note removed: "idk atp"
- note removed: "vbat to 9v (dji o3 maybe other stuff??)"
- moved on the sheet: C1, C11, C13, C14, C15, C16, C21, C22, C23, C24, C26, C27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

Commit message: finished routinnnn
:3
Parts:
- added C48: 10uf, Capacitor_SMD:C_0805_2012Metric, symbol Device:C
Connections:
- net GND: now also C48.2
- net VDD: now also C48.1
Other:
- moved on the sheet: C44
Changed lines of the file:
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@@
 	)
 	(junction
+		(at 187.96 27.94)
+		(diameter 0)
+		(color 0 0 0 0)
+	)
+	(junction
 		(at 382.27 223.52)
 		(diameter 0)
@@
 	)
 	(junction
+		(at 187.96 35.56)
+		(diameter 0)
+		(color 0 0 0 0)
+	)
+	(junction
 		(at 396.24 220.98)
 		(diameter 0)
@@
 	(wire
 		(pts
+			(xy 201.93 35.56) (xy 187.96 35.56)
+		)
+		(stroke
+			(width 0)
+			(type default)
+		)
+	)
+	(wire
+		(pts
 			(xy 104.14 35.56) (xy 90.17 35.56)
 		)
@@
 	(wire
 		(pts
+			(xy 201.93 27.94) (xy 187.96 27.94)
+		)
+		(stroke
+			(width 0)
+			(type default)
+		)
+	)
+	(wire
+		(pts
 			(xy 110.49 99.06) (xy 97.79 99.06)
 		)
@@
 	(symbol
 		(lib_id "Device:C")
-		(at 69.85 31.75 0)
-		(mirror y)
+		(at 201.93 31.75 0)
 		(unit 1)
 		(exclude_from_sim no)
@@
 		(dnp no)
 		(property "Reference" "C44"
-			(at 66.04 30.4799 0)
+			(at 205.74 30.4799 0)
 			(effects
 				(font
@@
 		)
 		(property "Value" "10uf"
-			(at 66.04 33.0199 0)
+			(at 205.74 33.0199 0)
 			(effects
 				(font
@@
 		)
 		(property "Footprint" "Capacitor_SMD:C_0805_2012Metric"
-			(at 68.8848 35.56 0)
+			(at 202.8952 35.56 0)
 			(effects
 				(font
@@
 		)
 		(property "Datasheet" "~"
-			(at 69.85 31.75 0)
+			(at 201.93 31.75 0)
 			(effects
 				(font
@@
 		)
 		(property "Description" "Unpolarized capacitor"
-			(at 69.85 31.75 0)
+			(at 201.93 31.75 0)
 			(effects
 				(font
@@
 		)
 		(property "LCSC Part" "C91185"
-			(at 69.85 31.75 0)
+			(at 201.93 31.75 0)
 			(effects
 				(font
@@
 					(unit 1)
 				)
+			)
+		)
+	)
+	(symbol
+		(lib_id "Device:C")
+		(at 69.85 31.75 0)
+		(mirror y)
+		(unit 1)
+		(exclude_from_sim no)
+		(in_bom yes)
+		(on_board yes)
+		(dnp no)
+		(property "Reference" "C48"
+			(at 66.04 30.4799 0)
+			(effects
+				(font
+					(size 1.27 1.27)
+				)
+				(justify left)
+			)
+		)
+		(property "Value" "10uf"
+			(at 66.04 33.0199 0)
+			(effects
+				(font
+					(size 1.27 1.27)
+				)
+				(justify left)
+			)
+		)
+		(property "Footprint" "Capacitor_SMD:C_0805_2012Metric"
+			(at 68.8848 35.56 0)
+			(effects
+				(font
+					(size 1.27 1.27)
+				)
+				(hide yes)
+			)
+		)
+		(property "Datasheet" "~"
+			(at 69.85 31.75 0)
+			(effects
+				(font
+					(size 1.27 1.27)
+				)
+				(hide yes)
+			)
+		)
+		(property "Description" "Unpolarized capacitor"
+			(at 69.85 31.75 0)
+			(effects
+				(font
+					(size 1.27 1.27)
+				)
+				(hide yes)
+			)
+		)
+		(property "LCSC Part" "C91185"
+			(at 69.85 31.75 0)
+			(effects
+				(font
+					(size 1.27 1.27)
+				)
+				(hide yes)
+			)
+		)
+		(pin "1"
+		)
+		(pin "2"
+		)
+		(instances
+			(project "drone"
+				(path "/16fe0d4b-7474-4548-8065-39d6508639c6"
+					(reference "C48")
+					(unit 1)
+				)

Commit message: a
Parts:
- added J30, J31, J32: Conn_01x01, TestPoint:TestPoint_Pad_1.0x1.0mm, symbol Connector_Generic:Conn_01x01
- C1, C11, C12, C15, C16, C21, C22, C25, C26, C29, C35, C37, C38, C4, C41, C42, C43, C45, C46, C49, C5, C51, C6: value 100nf -> 100n
- C10, C9: LCSC Part (none) -> C526978
- C13, C14, C23, C24: value 1uf -> 1u
- C17, C33, C8: LCSC Part (none) -> C1525
- C18, C20, C30, C36: LCSC Part (none) -> C602037
- C19, C34: LCSC Part (none) -> C138687
- C2, C3, C31, C7: LCSC Part (none) -> C50767367
- C27, C47: value 2.2uf -> 2.2u
- C28, C32, C39, C40: value 1uf -> 1u; LCSC Part C52923 -> C913556
- C44, C48: value 10uf -> 10u
- J1, J10, J11, J13, J14, J15, J16, J17, J18, J19, J20, J21, J22, J23, J24, J25, J26, J27, J28, J29, J3, J4, J5, J6, J7, J8, J9: LCSC Part (none) -> x
- L1: LCSC Part (none) -> C2879700
- R1, R13, R2, R20, R22, R23, R24, R27, R28, R29, R3, R30, R4: LCSC Part C25744 -> C190095
- R10, R5, R7, R9: LCSC Part (none) -> C445619
- R11, R19, R21: LCSC Part C11702 -> C445596
- R12: LCSC Part C1166 -> C445619
- R14, R6: LCSC Part (none) -> C852664
- R25: LCSC Part (none) -> x(shunt); now left out of the parts list
- R26: LCSC Part (none) -> C445596
- R8: LCSC Part (none) -> C427200
- U3: LCSC Part (none) -> C2441427
- U4: LCSC Part (none) -> C39843328
- U8: LCSC Part (none) -> C83291
- Y1: LCSC Part (none) -> C20625731
Connections:
- net GND: no longer U5.9 (INT2/FSYNC/CLKIN)
- net LED_1: now also U4.13 (GPIO14); no longer U4.11 (GPIO12)
- net LED_2: now also J30.1 (Pin_1); no longer U4.12 (GPIO13)
- net LED_3: now also J31.1 (Pin_1); no longer U4.13 (GPIO14)
- net LED_4: now also J32.1 (Pin_1); no longer U4.14 (GPIO15)
- net IMU_CLKIN: now reaches U4.27 (GPIO26)
- net IMU_CLKIN: now also U5.9 (INT2/FSYNC/CLKIN)
