File: src/hardware/esc/esc.kicad_pcb (KiCad board)
At the start: 6 copper layers, 40 x 40 mm, 222 parts, among them J1 Conn_01x03, J10 Conn_01x01, J11 Conn_01x01, J12 Conn_01x01, J2 Conn_01x03, J21 Conn_01x03, J3 Conn_01x03, J4 Conn_01x08, J5 Conn_01x01, J6 Conn_01x01, J7 Conn_01x01, J8 Conn_01x01, J9 Conn_01x01, Q1 NMOS, Q10 NMOS, Q11 NMOS, Q12 NMOS, Q13 NMOS, Q14 NMOS, Q15 NMOS, Q16 NMOS, Q17 NMOS, Q18 NMOS, Q19 NMOS, Q2 NMOS, Q20 NMOS, Q21 NMOS, Q22 NMOS, Q23 NMOS, Q24 NMOS, Q3 NMOS, Q4 NMOS, Q5 NMOS, Q6 NMOS, Q7 NMOS, Q8 NMOS, Q9 NMOS, U1 STM32L431K_B-C_Ux, U10 STM32L431K_B-C_Ux, U11 FD6288Q_C328453, U12 INA240A1PW, U13 STM32L431K_B-C_Ux, U14 FD6288Q_C328453, U15 INA240A1PW, U2 INA240A1PW, U3 FD6288Q_C328453, U4 TPS5430DDA, U5 AMS1117-3.3, U6 AMS1117-3.3, U7 STM32L431K_B-C_Ux, U8 FD6288Q_C328453, U9 INA240A1PW

Commit message: wip
Parts:
- removed C29, C43: 100n, Capacitor_SMD:C_0402_1005Metric
- removed C48, C72: 10u, Capacitor_SMD:C_1210_3225Metric
- removed C7: 68uF, Capacitor_Tantalum_SMD:CP_EIA-6032-28_Kemet-C
- removed D4: SS26, Diode_SMD:D_SMA
- removed U12, U15, U9: INA240A1PW, Package_SO:TSSOP-8_4.4x3mm_P0.65mm
- removed U6: AMS1117-3.3, Package_TO_SOT_SMD:SOT-223-3_TabPin2
- added C73: 1u, Capacitor_SMD:C_0402_1005Metric, B.Cu at (162.7, 57.9)
- added C74: 2.2u, Capacitor_SMD:C_0402_1005Metric, B.Cu at (162.7, 58.8)
- added C75: 100n, Capacitor_SMD:C_0402_1005Metric, B.Cu at (163.5, 63.6)
- added C76: 2.2u, Capacitor_SMD:C_0603_1608Metric, B.Cu at (169.7, 60.7)
- added C77: 5.1p, Capacitor_SMD:C_0402_1005Metric, B.Cu at (164.2, 55.0)
- added C78: 10u, Capacitor_SMD:C_0805_2012Metric, B.Cu at (165.8, 64.3)
- added C79: 10u, Capacitor_SMD:C_0805_2012Metric, B.Cu at (162.0, 63.4)
- added R32: 105k, Resistor_SMD:R_0402_1005Metric, B.Cu at (168.3, 55.5)
- added R51: 36.5k, Resistor_SMD:R_0402_1005Metric, B.Cu at (162.7, 56.9)
- added R71: 10k, Resistor_SMD:R_0402_1005Metric, F.Cu at (44.5, 48.8)
- added R72: 10k, Resistor_SMD:R_0402_1005Metric, F.Cu at (44.5, 50.8)
- added R84: 10k, Resistor_SMD:R_0402_1005Metric, F.Cu at (47.4, 46.8)
- added R85: 10k, Resistor_SMD:R_0402_1005Metric, F.Cu at (47.4, 48.8)
- C14, C20, C24, C31, C34, C4, C45, C52, C59, C60, C61, C62, C63, C64, C65, C66, C67, C68, C69, C70, C9: footprint Capacitor_SMD:C_1210_3225Metric -> Capacitor_SMD:C_0805_2012Metric
- C15, C38: footprint Capacitor_SMD:C_1210_3225Metric -> Capacitor_SMD:C_0805_2012Metric; moved to B.Cu
- C16: value 10n -> 470n; moved to B.Cu
- C39, R12, R13, R16, R17, R19, R20, R31, R38, R39, R40, R41, R5, R59, R60, R61, R7, R79, R80, R81, R9, U11, U14: moved to B.Cu
- D1, D10, D11, D12, D13, D14, D2, D3, D6, D7, D8, D9: value 1N4148W -> 1N4148WT; footprint Diode_SMD:D_SOD-123 -> Diode_SMD:D_SOD-523
- J1, J21, R4, REF** (x4), U3: moved to F.Cu
- J10, J11, J12, J5, J6, J7, J8, J9: footprint TestPoint:TestPoint_Pad_1.0x1.0mm -> TestPoint:TestPoint_Pad_D1.0mm
- J4: value Conn_01x08 -> Conn_01x08_MountingPin
- L1: footprint Inductor_SMD:L_Chilisin_BMRF00101040 -> footprint_lib:inductor FANGCHENG FC-ALX 5050D-150MT
- Q1, Q13, Q14, Q15, Q19, Q20, Q21, Q3, Q5, Q7, Q8, Q9: value NMOS -> RS60N80UHG; moved to F.Cu
- Q10, Q11, Q12, Q16, Q17, Q18, Q2, Q22, Q23, Q24, Q4, Q6: value NMOS -> RS60N80UHG; moved to B.Cu
- R10: value 10k -> 100k; moved to B.Cu
- R11: value 1.58k -> 12.4k; moved to B.Cu
- R2, R42, R62, R82: value 2mr -> 1mr; footprint Resistor_SMD:R_2010_5025Metric -> Resistor_SMD:R_1210_3225Metric; moved to B.Cu
- U1, U7: value STM32L431K_B-C_Ux -> STM32F051K8U6; moved to B.Cu
- U10, U13: value STM32L431K_B-C_Ux -> STM32F051K8U6
- U2: value INA240A1PW -> INA4180A2; footprint Package_SO:TSSOP-8_4.4x3mm_P0.65mm -> Package_SO:TSSOP-14_4.4x5mm_P0.65mm
- U4: value TPS5430DDA -> LM76003/2; footprint Package_SO:TI_SO-PowerPAD-8_ThermalVias -> Package_DFN_QFN:Texas_RNP0030B_WQFN-30-1EP_4x6mm_P0.5mm_EP1.8x4.5mm_ThermalVias; moved to B.Cu
- U5: value AMS1117-3.3 -> LDL212PV33R; footprint Package_TO_SOT_SMD:SOT-223-3_TabPin2 -> easyeda2kicad:DFN-6_L2.0-W2.0-P0.50-BL-EP1.45
- moved U5 220.7 mm to (33.1, 59.7)
- moved D10 177.7 mm to (176.3, -46.9)
- moved D11 177.7 mm to (182.1, -57.0)
- moved D9 177.7 mm to (176.3, -50.3)
- moved C13 173.6 mm to (234.9, 75.9)
- moved D3 171.8 mm to (222.5, 64.6)
- moved U4 152.8 mm to (166.3, 59.7)
- moved R23 150.4 mm to (80.6, 63.9)
- moved C34 149.6 mm to (68.0, 63.4)
- moved L1 147.9 mm to (162.4, 62.5)
- moved C42 140.6 mm to (190.9, -44.0)
- moved C20 135.0 mm to (68.0, 57.4)
- moved C40 132.0 mm to (186.9, -39.0)
- moved C41 132.0 mm to (186.9, -36.5)
- moved C9 125.7 mm to (148.8, 63.4), turned to -90 degrees
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Connections:
- C16 pad 2: Net-(D4-K) -> Net-(C16-Pad2)
- J4 pad MP: (no net) -> GND
- L1 pad 1: Net-(D4-K) -> Net-(C16-Pad2)
- Q10 pad S: Net-(U9-+) -> /curr2+
- Q11 pad S: Net-(U9-+) -> /curr2+
- Q12 pad S: Net-(U9-+) -> /curr2+
- Q16 pad S: Net-(U12-+) -> /curr3+
- Q17 pad S: Net-(U12-+) -> /curr3+
- Q18 pad S: Net-(U12-+) -> /curr3+
- Q2 pad S: Net-(U2-+) -> /curr1+
- Q22 pad S: Net-(U15-+) -> /curr4+
- Q23 pad S: Net-(U15-+) -> /curr4+
- Q24 pad S: Net-(U15-+) -> /curr4+
- Q4 pad S: Net-(U2-+) -> /curr1+
- Q6 pad S: Net-(U2-+) -> /curr1+
- R10 pad 1: Net-(U4-VSENSE) -> Net-(U4-FB)
- R11 pad 2: Net-(U4-VSENSE) -> Net-(U4-FB)
- R2 pad 1: Net-(U2-+) -> /curr1+
- R2 pad 2: GND -> /curr1-
- R42 pad 1: Net-(U9-+) -> /curr2+
- R42 pad 2: GND -> /curr2-
- R62 pad 1: Net-(U12-+) -> /curr3+
- R62 pad 2: GND -> /curr3-
- R82 pad 1: Net-(U15-+) -> /curr4+
- R82 pad 2: GND -> /curr4-
- U1 pad 12: /V_SENS1 -> /V_SENS
- U1 pad 31: unconnected-(U1-PH3-Pad31) -> Net-(U1-PH3)
- U10 pad 12: /V_SENS3 -> /V_SENS
- U10 pad 31: unconnected-(U10-PH3-Pad31) -> Net-(U10-PH3)
- U13 pad 12: /V_SENS4 -> /V_SENS
- U13 pad 31: unconnected-(U13-PH3-Pad31) -> Net-(U13-PH3)
- U2 pad 1: GND -> Net-(R83-Pad1)
- U2 pad 2: Net-(U2-+) -> /curr4-
- U2 pad 3: GND -> /curr4+
- U2 pad 4: GND -> VCC
- U2 pad 5: VCC -> /curr2+
- U2 pad 6: GND -> /curr2-
- U2 pad 7: GND -> Net-(R43-Pad1)
- U4 pad 1: Net-(U4-BOOT) -> Net-(C16-Pad2)
- U4 pad 2: unconnected-(U4-NC-Pad2) -> Net-(C16-Pad2)
- U4 pad 3: unconnected-(U4-NC-Pad3) -> Net-(C16-Pad2)
- U4 pad 4: Net-(U4-VSENSE) -> Net-(C16-Pad2)
- U4 pad 5: +BATT -> Net-(C16-Pad2)
- U4 pad 6: GND -> Net-(U4-BOOT)
- U4 pad 7: +BATT -> unconnected-(U4-NC-Pad7)
- U4 pad 8: Net-(D4-K) -> Net-(U4-VCC)
- U4 pad 9: GND -> +9V
- U5 pad 3: +9V -> VCC
- U7 pad 12: /V_SENS2 -> /V_SENS
- U7 pad 31: unconnected-(U7-PH3-Pad31) -> Net-(U7-PH3)
Routing:
- added copper zone on B.Cu, net GND
- added copper zone on F.Cu, net GND
- added copper zone on In1.Cu, net GND
- added copper zone on In3.Cu, net GND
Other:
- board size 40 x 40 mm -> 50.9 x 40 mm

Commit message: a
Parts:
- removed R46: 10k, Resistor_SMD:R_0402_1005Metric
- added ?: , , F.Cu at (168.6, 27.1)
- added ?: , , F.Cu at (156.1, 27.1)
- added J13: Conn_02x05_Odd_Even, Connector_PinHeader_1.00mm:PinHeader_2x05_P1.00mm_Vertical, F.Cu at (153.1, 18.1)
- added J14: Conn_02x05_Odd_Even, Connector_PinHeader_1.00mm:PinHeader_2x05_P1.00mm_Vertical, F.Cu at (167.6, 18.1)
- added J15: Conn_02x07_Odd_Even, Connector_PinHeader_1.00mm:PinHeader_2x07_P1.00mm_Vertical, F.Cu at (156.8, 56.9)
- added J16: Conn_01x02, Connector_PinHeader_1.00mm:PinHeader_1x02_P1.00mm_Vertical, F.Cu at (152.3, 55.4)
- added J17: Conn_01x02, Connector_PinHeader_1.00mm:PinHeader_1x02_P1.00mm_Vertical, F.Cu at (144.7, 55.4)
- added J18: Conn_01x02, Connector_PinHeader_1.00mm:PinHeader_1x02_P1.00mm_Vertical, F.Cu at (144.7, 64.4)
- added J19: Conn_02x05_Odd_Even, Connector_PinHeader_1.00mm:PinHeader_2x05_P1.00mm_Vertical, F.Cu at (153.8, 55.4)
- added J20: Conn_02x05_Odd_Even, Connector_PinHeader_1.00mm:PinHeader_2x05_P1.00mm_Vertical, F.Cu at (139.3, 55.4)
- added J22: Conn_01x02, Connector_PinHeader_1.00mm:PinHeader_1x02_P1.00mm_Vertical, F.Cu at (152.3, 64.4)
- added J25: Conn_01x02, Connector_PinHeader_1.00mm:PinHeader_1x02_P1.00mm_Vertical, F.Cu at (158.5, 18.1)
- added J26: Conn_01x02, Connector_PinHeader_1.00mm:PinHeader_1x02_P1.00mm_Vertical, F.Cu at (166.1, 17.1)
- added J27: Conn_02x05_Odd_Even, Connector_PinHeader_1.00mm:PinHeader_2x05_P1.00mm_Vertical, F.Cu at (157.8, 64.4)
- added J28: Conn_02x05_Odd_Even, Connector_PinHeader_1.00mm:PinHeader_2x05_P1.00mm_Vertical, F.Cu at (143.3, 64.4)
- added J29: Conn_02x04_Odd_Even, Connector_PinHeader_1.00mm:PinHeader_2x04_P1.00mm_Vertical, B.Cu at (171.6, 19.6)
- added U6: INA2180A1, Package_SON:WSON-8-1EP_2x2mm_P0.5mm_EP0.9x1.6mm, F.Cu at (162.5, 17.7)
- C17, C20, C30, C31, C35, C37, C40, C41, C42, C53, C54, C55, C56, C58, C69, C70, C8, D10, D11, D12, D13, D14, D9, R14, R15, R18, R21, R22, R23, R28, R29, R3, R30, R33, R34, R35, R43, R45, R47, R53, R65, R66, R69, R72, R73, U5: moved to B.Cu
- C24, C38, C9: footprint Capacitor_SMD:C_0805_2012Metric -> Capacitor_SMD:C_0603_1608Metric
- C52: footprint Capacitor_SMD:C_0805_2012Metric -> Capacitor_SMD:C_0603_1608Metric; moved to B.Cu
- C79, U1, U7: moved to F.Cu
- U2: value INA4180A2 -> INA2180A1; footprint Package_SO:TSSOP-14_4.4x5mm_P0.65mm -> Package_SON:WSON-8-1EP_2x2mm_P0.5mm_EP0.9x1.6mm
- moved R14 1316.5 mm to (-1140.0, 232.3)
- moved R15 1316.5 mm to (-1140.0, 233.2)
- moved R18 1316.5 mm to (-1140.0, 234.2)
- moved R12 1313.9 mm to (-1143.3, 233.7)
- moved R13 1313.9 mm to (-1143.3, 235.6)
- moved R16 1312.0 mm to (-1142.4, 235.6)
- moved R17 1312.0 mm to (-1142.4, 233.7)
- moved R19 1310.2 mm to (-1141.4, 235.6)
- moved R20 1310.2 mm to (-1141.4, 233.7)
- moved C13 1309.5 mm to (-1071.7, 163.8)
- moved D3 1309.5 mm to (-1084.1, 152.5)
- moved U3 1292.8 mm to (-1138.7, 113.6), turned to 90 degrees
- moved U8 1288.9 mm to (-1145.8, 114.0)
- moved U2 1288.4 mm to (-1127.5, 93.5), turned to -90 degrees
- moved U1 1286.2 mm to (-1133.5, 98.6)
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Connections:
- net /A_HIGH1 renamed /top/A_HIGH1
- net /A_HIGH2 renamed /top/A_HIGH2
- net /A_HIGH3 renamed /bottom/A_HIGH3
- net /A_HIGH4 renamed /bottom/A_HIGH4
- net /A_LOW1 renamed /top/A_LOW1
- net /A_LOW2 renamed /top/A_LOW2
- net /A_LOW3 renamed /bottom/A_LOW3
- net /A_LOW4 renamed /bottom/A_LOW4
- net /BEMF_A1 renamed /top/BEMF_A1
- net /BEMF_A2 renamed /top/BEMF_A2
- net /BEMF_A3 renamed /bottom/BEMF_A3
- net /BEMF_A4 renamed /bottom/BEMF_A4
- net /BEMF_B1 renamed /top/BEMF_B1
- net /BEMF_B2 renamed /top/BEMF_B2
- net /BEMF_B3 renamed /bottom/BEMF_B3
- net /BEMF_B4 renamed /bottom/BEMF_B4
- net /BEMF_C1 renamed /top/BEMF_C1
- net /BEMF_C2 renamed /top/BEMF_C2
- net /BEMF_C3 renamed /bottom/BEMF_C3
- net /BEMF_C4 renamed /bottom/BEMF_C4
- net /BEMF_COMMON1 renamed /top/BEMF_COMMON1
- net /BEMF_COMMON2 renamed /top/BEMF_COMMON2
- net /BEMF_COMMON3 renamed /bottom/BEMF_COMMON3
- net /BEMF_COMMON4 renamed /bottom/BEMF_COMMON4
- net /B_HIGH1 renamed /top/B_HIGH1
- net /B_HIGH2 renamed /top/B_HIGH2
- net /B_HIGH3 renamed /bottom/B_HIGH3
- net /B_HIGH4 renamed /bottom/B_HIGH4
- net /B_LOW1 renamed /top/B_LOW1
- net /B_LOW2 renamed /top/B_LOW2
- net /B_LOW3 renamed /bottom/B_LOW3
- net /B_LOW4 renamed /bottom/B_LOW4
- net /CURR1 renamed /top/CURR1
- net /CURR2 renamed /top/CURR2
- net /CURR3 renamed /bottom/CURR3
- net /CURR4 renamed /bottom/CURR4
- net /C_HIGH1 renamed /top/C_HIGH1
- net /C_HIGH2 renamed /top/C_HIGH2
- net /C_HIGH3 renamed /bottom/C_HIGH3
- net /C_HIGH4 renamed /bottom/C_HIGH4
- net /C_LOW1 renamed /top/C_LOW1
- net /C_LOW2 renamed /top/C_LOW2
- net /C_LOW3 renamed /bottom/C_LOW3
- net /C_LOW4 renamed /bottom/C_LOW4
- net /SWDCLK1 renamed /top/SWDCLK1
- net /SWDCLK2 renamed /top/SWDCLK2
- net /SWDCLK3 renamed /bottom/SWDCLK3
- net /SWDCLK4 renamed /bottom/SWDCLK4
- net /SWDIO1 renamed /top/SWDIO1
- net /SWDIO2 renamed /top/SWDIO2
- net /SWDIO3 renamed /bottom/SWDIO3
- net /SWDIO4 renamed /bottom/SWDIO4
- C10 pad 2: +9V -> /top/9v
- C11 pad 1: /MOT_A1 -> /top/MOT_A1
- C12 pad 1: /MOT_B1 -> /top/MOT_B1
- C13 pad 1: /MOT_C1 -> /top/MOT_C1
- C14 pad 1: VCC -> /top/vcc
- C18 pad 1: VCC -> /top/vcc
- C19 pad 1: VCC -> /top/vcc
- C2 pad 1: VCC -> /top/vcc
- C21 pad 1: VCC -> /top/vcc
- C22 pad 1: VCC -> /top/vcc
- C24 pad 1: +9V -> /top/9v
- C25 pad 2: +9V -> /top/9v
- C26 pad 1: /MOT_A2 -> /top/MOT_A2
- C27 pad 1: /MOT_B2 -> /top/MOT_B2
- C28 pad 1: /MOT_C2 -> /top/MOT_C2
- C3 pad 1: VCC -> /top/vcc
- C38 pad 1: +9V -> /bottom/9v
- C39 pad 2: +9V -> /bottom/9v
- C4 pad 1: VCC -> /top/vcc
- C40 pad 1: /MOT_A3 -> /bottom/MOT_A3
- C41 pad 1: /MOT_B3 -> /bottom/MOT_B3
- C42 pad 1: /MOT_C3 -> /bottom/MOT_C3
- C5 pad 1: VCC -> /top/vcc
- C52 pad 1: +9V -> /bottom/9v
- C53 pad 2: +9V -> /bottom/9v
- C54 pad 1: /MOT_A4 -> /bottom/MOT_A4
- C55 pad 1: /MOT_B4 -> /bottom/MOT_B4
- C56 pad 1: /MOT_C4 -> /bottom/MOT_C4
- C57 pad 1: VCC -> /top/vcc
- C6 pad 1: VCC -> /top/vcc
- C9 pad 1: +9V -> /top/9v
- D1 pad 2: +9V -> /top/9v
- D10 pad 2: +9V -> /bottom/9v
- D11 pad 2: +9V -> /bottom/9v
- D12 pad 2: +9V -> /bottom/9v
- D13 pad 2: +9V -> /bottom/9v
- D14 pad 2: +9V -> /bottom/9v
- D2 pad 2: +9V -> /top/9v
- D3 pad 2: +9V -> /top/9v
- D6 pad 2: +9V -> /top/9v
- D7 pad 2: +9V -> /top/9v
- D8 pad 2: +9V -> /top/9v
- D9 pad 2: +9V -> /bottom/9v
- J1 pad 1: /MOT_A2 -> /Powerstage/MOT_A2
- J1 pad 2: /MOT_B2 -> /Powerstage/MOT_B2
- J1 pad 3: /MOT_C2 -> /Powerstage/MOT_C2
- J2 pad 1: /MOT_A3 -> /Powerstage/MOT_A3
- J2 pad 2: /MOT_B3 -> /Powerstage/MOT_B3
- J2 pad 3: /MOT_C3 -> /Powerstage/MOT_C3
- J21 pad 1: /MOT_A1 -> /Powerstage/MOT_A1
- J21 pad 2: /MOT_B1 -> /Powerstage/MOT_B1
- J21 pad 3: /MOT_C1 -> /Powerstage/MOT_C1
- J3 pad 1: /MOT_A4 -> /Powerstage/MOT_A4
- J3 pad 2: /MOT_B4 -> /Powerstage/MOT_B4
- J3 pad 3: /MOT_C4 -> /Powerstage/MOT_C4
- J4 pad 3: /TELEMRX -> /Powerstage/TELEMRX
- J4 pad 4: /TELEMETRY -> /Powerstage/TELEMETRY
- J4 pad 5: /SIG_IN1 -> /Powerstage/SIG_IN1
- J4 pad 6: /SIG_IN2 -> /Powerstage/SIG_IN2
- J4 pad 7: /SIG_IN3 -> /Powerstage/SIG_IN3
- J4 pad 8: /SIG_IN4 -> /Powerstage/SIG_IN4
- Q1 pad S: /MOT_A1 -> /Powerstage/MOT_A1
- Q10 pad D: /MOT_A2 -> /Powerstage/MOT_A2
- Q10 pad S: /curr2+ -> /Powerstage/curr2+
- Q11 pad D: /MOT_B2 -> /Powerstage/MOT_B2
- Q11 pad S: /curr2+ -> /Powerstage/curr2+
- Q12 pad D: /MOT_C2 -> /Powerstage/MOT_C2
- Q12 pad S: /curr2+ -> /Powerstage/curr2+
- Q13 pad S: /MOT_A3 -> /Powerstage/MOT_A3
- Q14 pad S: /MOT_B3 -> /Powerstage/MOT_B3
- Q15 pad S: /MOT_C3 -> /Powerstage/MOT_C3
- Q16 pad D: /MOT_A3 -> /Powerstage/MOT_A3
- Q16 pad S: /curr3+ -> /Powerstage/curr3+
- Q17 pad D: /MOT_B3 -> /Powerstage/MOT_B3
- Q17 pad S: /curr3+ -> /Powerstage/curr3+
- Q18 pad D: /MOT_C3 -> /Powerstage/MOT_C3
- Q18 pad S: /curr3+ -> /Powerstage/curr3+
- Q19 pad S: /MOT_A4 -> /Powerstage/MOT_A4
- Q2 pad D: /MOT_A1 -> /Powerstage/MOT_A1
- Q2 pad S: /curr1+ -> /Powerstage/curr1+
- Q20 pad S: /MOT_B4 -> /Powerstage/MOT_B4
- Q21 pad S: /MOT_C4 -> /Powerstage/MOT_C4
- Q22 pad D: /MOT_A4 -> /Powerstage/MOT_A4
- Q22 pad S: /curr4+ -> /Powerstage/curr4+
- Q23 pad D: /MOT_B4 -> /Powerstage/MOT_B4
- Q23 pad S: /curr4+ -> /Powerstage/curr4+
- Q24 pad D: /MOT_C4 -> /Powerstage/MOT_C4
- Q24 pad S: /curr4+ -> /Powerstage/curr4+
- Q3 pad S: /MOT_B1 -> /Powerstage/MOT_B1
- Q4 pad D: /MOT_B1 -> /Powerstage/MOT_B1
- Q4 pad S: /curr1+ -> /Powerstage/curr1+
- Q5 pad S: /MOT_C1 -> /Powerstage/MOT_C1
- Q6 pad D: /MOT_C1 -> /Powerstage/MOT_C1
- Q6 pad S: /curr1+ -> /Powerstage/curr1+
- Q7 pad S: /MOT_A2 -> /Powerstage/MOT_A2
- Q8 pad S: /MOT_B2 -> /Powerstage/MOT_B2
- Q9 pad S: /MOT_C2 -> /Powerstage/MOT_C2
- R1 pad 1: /SIG_IN1 -> /top/SIG_IN1
- R13 pad 2: /MOT_A1 -> /top/MOT_A1
- R16 pad 2: /MOT_B1 -> /top/MOT_B1
- R19 pad 2: /MOT_C1 -> /top/MOT_C1
- R2 pad 1: /curr1+ -> /Powerstage/curr1+
- R2 pad 2: /curr1- -> /Powerstage/curr1-
- R21 pad 1: /V_SENS -> /Powerstage/V_SENS
- R22 pad 2: /V_SENS -> /Powerstage/V_SENS
- R24 pad 1: /SIG_IN2 -> /top/SIG_IN2
- R28 pad 2: /MOT_A2 -> /top/MOT_A2
- R29 pad 2: /MOT_B2 -> /top/MOT_B2
- R30 pad 2: /MOT_C2 -> /top/MOT_C2
- R36 pad 2: /GHA2 -> /Powerstage/GHA2
- R37 pad 2: /GHB2 -> /Powerstage/GHB2
- R38 pad 2: /GHC2 -> /Powerstage/GHC2
- R39 pad 2: /GLA2 -> /Powerstage/GLA2
- R4 pad 2: /GHA1 -> /Powerstage/GHA1
- R40 pad 2: /GLB2 -> /Powerstage/GLB2
- R41 pad 2: /GLC2 -> /Powerstage/GLC2
- R42 pad 1: /curr2+ -> /Powerstage/curr2+
- R42 pad 2: /curr2- -> /Powerstage/curr2-
- R44 pad 1: /SIG_IN3 -> /bottom/SIG_IN3
- R48 pad 2: /MOT_A3 -> /bottom/MOT_A3
- R49 pad 2: /MOT_B3 -> /bottom/MOT_B3
- R5 pad 2: /GLA1 -> /Powerstage/GLA1
- R50 pad 2: /MOT_C3 -> /bottom/MOT_C3
- R56 pad 2: /GHA3 -> /Powerstage/GHA3
- R57 pad 2: /GHB3 -> /Powerstage/GHB3
- R58 pad 2: /GHC3 -> /Powerstage/GHC3
- R59 pad 2: /GLA3 -> /Powerstage/GLA3
- R6 pad 2: /GHB1 -> /Powerstage/GHB1
- R60 pad 2: /GLB3 -> /Powerstage/GLB3
- R61 pad 2: /GLC3 -> /Powerstage/GLC3
- R62 pad 1: /curr3+ -> /Powerstage/curr3+
- R62 pad 2: /curr3- -> /Powerstage/curr3-
- R64 pad 1: /SIG_IN4 -> /bottom/SIG_IN4
- R68 pad 2: /MOT_A4 -> /bottom/MOT_A4
- R69 pad 2: /MOT_B4 -> /bottom/MOT_B4
- R7 pad 2: /GLB1 -> /Powerstage/GLB1
- R70 pad 2: /MOT_C4 -> /bottom/MOT_C4
- R76 pad 2: /GHA4 -> /Powerstage/GHA4
- R77 pad 2: /GHB4 -> /Powerstage/GHB4
- R78 pad 2: /GHC4 -> /Powerstage/GHC4
- R79 pad 2: /GLA4 -> /Powerstage/GLA4
- R8 pad 2: /GHC1 -> /Powerstage/GHC1
- R80 pad 2: /GLB4 -> /Powerstage/GLB4
- R81 pad 2: /GLC4 -> /Powerstage/GLC4
- R82 pad 1: /curr4+ -> /Powerstage/curr4+
- R82 pad 2: /curr4- -> /Powerstage/curr4-
- R9 pad 2: /GLC1 -> /Powerstage/GLC1
- U1 pad 1: VCC -> /top/vcc
- U1 pad 12: /V_SENS -> /top/V_SENS
- U1 pad 17: VCC -> /top/vcc
- U1 pad 29: /TELEMETRY -> /top/TELEMETRY
- U1 pad 30: /TELEMRX -> /top/TELEMRX
- U1 pad 5: VCC -> /top/vcc
- U10 pad 12: /V_SENS -> /bottom/V_SENS
- U10 pad 29: /TELEMETRY -> /bottom/TELEMETRY
- U10 pad 30: /TELEMRX -> /bottom/TELEMRX
- U11 pad 10: /GLB3 -> /bottom/GLB3
- U11 pad 11: /GLA3 -> /bottom/GLA3
- U11 pad 12: /MOT_C3 -> /bottom/MOT_C3
- U11 pad 13: /GHC3 -> /bottom/GHC3
- U11 pad 15: /MOT_B3 -> /bottom/MOT_B3
- U11 pad 16: /GHB3 -> /bottom/GHB3
- U11 pad 18: /MOT_A3 -> /bottom/MOT_A3
- U11 pad 19: /GHA3 -> /bottom/GHA3
- U11 pad 4: +9V -> /bottom/9v
- U11 pad 9: /GLC3 -> /bottom/GLC3
- U13 pad 12: /V_SENS -> /bottom/V_SENS
- U13 pad 29: /TELEMETRY -> /bottom/TELEMETRY
- U13 pad 30: /TELEMRX -> /bottom/TELEMRX
- U14 pad 10: /GLB4 -> /bottom/GLB4
- U14 pad 11: /GLA4 -> /bottom/GLA4
- U14 pad 12: /MOT_C4 -> /bottom/MOT_C4
- U14 pad 13: /GHC4 -> /bottom/GHC4
- U14 pad 15: /MOT_B4 -> /bottom/MOT_B4
- U14 pad 16: /GHB4 -> /bottom/GHB4
- U14 pad 18: /MOT_A4 -> /bottom/MOT_A4
- U14 pad 19: /GHA4 -> /bottom/GHA4
- U14 pad 4: +9V -> /bottom/9v
- U14 pad 9: /GLC4 -> /bottom/GLC4
- U2 pad 1: Net-(R83-Pad1) -> Net-(R3-Pad1)
- U2 pad 2: /curr4- -> /top/curr1-
- U2 pad 3: /curr4+ -> /top/curr1+
- U2 pad 4: VCC -> GND
- U2 pad 5: /curr2+ -> /top/curr2+
- U2 pad 6: /curr2- -> /top/curr2-
- U2 pad 8: Net-(R3-Pad1) -> unconnected-(U2C-VCC-Pad8)
- U2 pad 9: /curr1- -> GND
- U3 pad 10: /GLB1 -> /top/GLB1
- U3 pad 11: /GLA1 -> /top/GLA1
- U3 pad 12: /MOT_C1 -> /top/MOT_C1
- U3 pad 13: /GHC1 -> /top/GHC1
- U3 pad 15: /MOT_B1 -> /top/MOT_B1
- U3 pad 16: /GHB1 -> /top/GHB1
- U3 pad 18: /MOT_A1 -> /top/MOT_A1
- U3 pad 19: /GHA1 -> /top/GHA1
- U3 pad 4: +9V -> /top/9v
- U3 pad 9: /GLC1 -> /top/GLC1
- U7 pad 1: VCC -> /top/vcc
- U7 pad 12: /V_SENS -> /top/V_SENS
- U7 pad 17: VCC -> /top/vcc
- U7 pad 29: /TELEMETRY -> /top/TELEMETRY
- U7 pad 30: /TELEMRX -> /top/TELEMRX
- U7 pad 5: VCC -> /top/vcc
- U8 pad 10: /GLB2 -> /top/GLB2
- U8 pad 11: /GLA2 -> /top/GLA2
- U8 pad 12: /MOT_C2 -> /top/MOT_C2
- U8 pad 13: /GHC2 -> /top/GHC2
- U8 pad 15: /MOT_B2 -> /top/MOT_B2
- U8 pad 16: /GHB2 -> /top/GHB2
- U8 pad 18: /MOT_A2 -> /top/MOT_A2
- U8 pad 19: /GHA2 -> /top/GHA2
- U8 pad 4: +9V -> /top/9v
- U8 pad 9: /GLC2 -> /top/GLC2
Routing:
- net +BATT: track 0.00 -> 113.1 mm, vias 0 -> 8
- net VCC: track 0.00 -> 75.2 mm, vias 0 -> 6
- net +9V: track 0.00 -> 41.1 mm, vias 0 -> 7
- net /Powerstage/TELEMETRY: track 0.00 -> 28.7 mm, vias 0 -> 1
- net /Powerstage/curr3+: track 0.00 -> 27.7 mm
- net /bottom/TELEMETRY: track 0.00 -> 26.0 mm, vias 0 -> 2
- net /Powerstage/curr4+: track 0.00 -> 25.6 mm
- net /Powerstage/SIG_IN1: track 0.00 -> 24.3 mm, vias 0 -> 1
- net /bottom/V_SENS: track 0.00 -> 23.2 mm, vias 0 -> 2
- net /bottom/TELEMRX: track 0.00 -> 22.1 mm, vias 0 -> 1
- net /Powerstage/TELEMRX: track 0.00 -> 20.9 mm, vias 0 -> 1
- net /Powerstage/MOT_C2: track 0.00 -> 20.6 mm, vias 0 -> 63
- net /Powerstage/SIG_IN2: track 0.00 -> 20.4 mm, vias 0 -> 1
- net /Powerstage/GHC2: track 0.00 -> 17.8 mm, vias 0 -> 1
- net /Powerstage/GHA4: track 0.00 -> 17.1 mm, vias 0 -> 1
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- added copper zone on F.Cu, net +9V
- added copper zone on B.Cu, net +BATT
- added copper zone on F.Cu, net +BATT
- added copper zone on In2.Cu, net +BATT
- added copper zone on In4.Cu, net +BATT
- added copper zone on B.Cu, net /Powerstage/MOT_A1
- added copper zone on F.Cu, net /Powerstage/MOT_A1
- added copper zone on B.Cu, net /Powerstage/MOT_A2
- added copper zone on F.Cu, net /Powerstage/MOT_A2
- added copper zone on B.Cu, net /Powerstage/MOT_A3
- added copper zone on F.Cu, net /Powerstage/MOT_A3
- added copper zone on B.Cu, net /Powerstage/MOT_A4
- added copper zone on F.Cu, net /Powerstage/MOT_A4
- added copper zone on B.Cu, net /Powerstage/MOT_B1
- added copper zone on F.Cu, net /Powerstage/MOT_B1
- added copper zone on B.Cu, net /Powerstage/MOT_B2
- added copper zone on F.Cu, net /Powerstage/MOT_B2
- added copper zone on B.Cu, net /Powerstage/MOT_B3
- added copper zone on F.Cu, net /Powerstage/MOT_B3
- added copper zone on B.Cu, net /Powerstage/MOT_B4
- added copper zone on F.Cu, net /Powerstage/MOT_B4
- added copper zone on B.Cu, net /Powerstage/MOT_C1
- added copper zone on F.Cu, net /Powerstage/MOT_C1
- added copper zone on B.Cu, net /Powerstage/MOT_C2
- added copper zone on F.Cu, net /Powerstage/MOT_C2
- added copper zone on B.Cu, net /Powerstage/MOT_C3
- added copper zone on F.Cu, net /Powerstage/MOT_C3
- added copper zone on B.Cu, net /Powerstage/MOT_C4
- added copper zone on F.Cu, net /Powerstage/MOT_C4
- added copper zone on B.Cu, net /Powerstage/curr1+
- added copper zone on B.Cu, net /Powerstage/curr2+
- added copper zone on B.Cu, net /Powerstage/curr3+
- added copper zone on B.Cu, net /bottom/curr4+
- added copper zone on B.Cu, net Net-(C16-Pad2)
Other:
- board size 50.9 x 40 mm -> 50.9 x 63.7 mm

Commit message: a
Parts:
- removed C1, C10, C18, C19, C22, C23, C25, C3, C5, C57, C6: 100n, Capacitor_SMD:C_0402_1005Metric
- removed C11, C12, C13, C2, C21, C26, C27, C28: 1u, Capacitor_SMD:C_0603_1608Metric
- removed C14, C4: 10u, Capacitor_SMD:C_0805_2012Metric
- removed C24, C9: 10u, Capacitor_SMD:C_0603_1608Metric
- removed C30, C8: 10n, Capacitor_SMD:C_0402_1005Metric
- removed D1, D2, D3, D6, D7, D8: 1N4148WT, Diode_SMD:D_SOD-523
- removed J5, J6, J7, J8: Conn_01x01, TestPoint:TestPoint_Pad_D1.0mm
- removed R1, R12, R17, R20, R24, R3, R33, R34, R35, R43: 1k, Resistor_SMD:R_0402_1005Metric
- removed R13, R14, R15, R16, R18, R19, R25, R26, R27, R28, R29, R30, R84, R85: 10k, Resistor_SMD:R_0402_1005Metric
- removed U1, U7: STM32F051K8U6, Package_DFN_QFN:QFN-32-1EP_5x5mm_P0.5mm_EP3.45x3.45mm
- removed U2: INA2180A1, Package_SON:WSON-8-1EP_2x2mm_P0.5mm_EP0.9x1.6mm
- removed U3, U8: FD6288Q_C328453, easyeda2kicad:QFN-24_L4.0-W4.0-P0.50-BL-EP2.6
- added C72: 10u, Capacitor_SMD:C_0603_1608Metric, B.Cu at (148.9, 62.6)
- added R46: 10k, Resistor_SMD:R_0402_1005Metric, F.Cu at (143.1, 53.0)
- C37, R45, R47, R66, R69, R72: moved to F.Cu
- R55: moved to B.Cu
- moved L1 85.4 mm to (77.1, 63.0)
- moved C20 85.4 mm to (75.3, 63.5)
- moved C77 85.4 mm to (78.8, 57.1)
- moved C78 85.4 mm to (78.5, 65.5)
- moved D15 85.4 mm to (46.2, 61.0)
- moved D5 85.4 mm to (75.9, 56.7)
- moved J1 85.4 mm to (56.8, 78.5)
- moved J19 85.4 mm to (68.4, 56.6)
- moved J2 85.4 mm to (68.7, 43.4)
- moved J27 85.4 mm to (72.4, 65.6)
- moved J4 85.4 mm to (85.2, 61.1)
- moved Q12 85.4 mm to (48.6, 69.0)
- moved Q13 85.4 mm to (65.4, 49.8)
- moved Q15 85.4 mm to (77.2, 53.0)
- moved Q18 85.4 mm to (77.2, 53.0)
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Connections:
- C38 pad 1: /bottom/9v -> +9V
- C39 pad 2: /bottom/9v -> +9V
- C52 pad 1: /bottom/9v -> +9V
- C53 pad 2: /bottom/9v -> +9V
- D10 pad 2: /bottom/9v -> +9V
- D11 pad 2: /bottom/9v -> +9V
- D12 pad 2: /bottom/9v -> +9V
- D13 pad 2: /bottom/9v -> +9V
- D14 pad 2: /bottom/9v -> +9V
- D9 pad 2: /bottom/9v -> +9V
- U11 pad 4: /bottom/9v -> +9V
- U14 pad 4: /bottom/9v -> +9V
Routing:
- net +9V: track 41.1 -> 105.1 mm, vias 7 -> 13
- net VCC: track 75.2 -> 92.3 mm, vias 6 -> 8
- net GND: track 0.00 -> 16.8 mm, vias 122 -> 159
- net /bottom/MOT_A3: track 9.65 -> 24.4 mm, vias 1 -> 2
- net /bottom/BEMF_B3: track 2.55 -> 15.3 mm, vias 0 -> 2
- net /bottom/MOT_C3: track 6.01 -> 18.8 mm, vias 0 -> 2
- net /bottom/GHA3: track 2.12 -> 14.4 mm
- net /bottom/MOT_B4: track 4.06 -> 14.6 mm
- net /bottom/GHA4: track 7.52 -> 16.9 mm, vias 0 -> 1
- net /bottom/BEMF_COMMON3: track 6.72 -> 16.0 mm, vias 1 -> 3
- net /bottom/V_SENS: track 23.2 -> 31.3 mm, vias 2 -> 4
- net Net-(U10-NRST): track 9.98 -> 2.71 mm, vias 1 -> 0
- net /bottom/9v: track 7.14 -> 0.00 mm
- net /Powerstage/GHC3: track 10.1 -> 16.4 mm, vias 0 -> 1
- net /bottom/CURR3: track 0.00 -> 5.38 mm
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- added copper zone on In2.Cu, net GND
- added copper zone on In4.Cu, net GND
Other:
- board size 50.9 x 63.7 mm -> 112 x 40 mm
