File: src/hardware/esc/esc.kicad_sch (KiCad schematic)
At the start: 217 parts, among them J1 Conn_01x03, J10 Conn_01x01, J11 Conn_01x01, J12 Conn_01x01, J2 Conn_01x03, J21 Conn_01x03, J3 Conn_01x03, J4 Conn_01x08, J5 Conn_01x01, J6 Conn_01x01, J7 Conn_01x01, J8 Conn_01x01, J9 Conn_01x01, Q1 NMOS, Q10 NMOS, Q11 NMOS, Q12 NMOS, Q13 NMOS, Q14 NMOS, Q15 NMOS, Q16 NMOS, Q17 NMOS, Q18 NMOS, Q19 NMOS, Q2 NMOS, Q20 NMOS, Q21 NMOS, Q22 NMOS, Q23 NMOS, Q24 NMOS, Q3 NMOS, Q4 NMOS, Q5 NMOS, Q6 NMOS, Q7 NMOS, Q8 NMOS, Q9 NMOS, U10 STM32L431CCUx, U11 FD6288Q_C328453, U12 INA240A1PW, U13 STM32L431CCUx, U14 FD6288Q_C328453, U15 INA240A1PW, U16 STM32L431K_B-C_Ux, U2 INA240A1PW, U3 FD6288Q_C328453, U4 TPS5430DDA, U5 AMS1117-3.3, U6 AMS1117-3.3, U7 STM32L431CCUx, U8 FD6288Q_C328453, U9 INA240A1PW

Commit message: update sch
fixed wrong mcu package
+ i suppose gitignore doing its thing
Parts:
- removed C20, C34, C48, C7: 100n, Capacitor_SMD:C_0402_1005Metric, symbol Device:C
- removed U10, U13, U7: STM32L431CCUx, Package_DFN_QFN:QFN-48-1EP_7x7mm_P0.5mm_EP5.6x5.6mm, symbol MCU_ST_STM32L4:STM32L431CCUx
- added U10, U13, U7: STM32L431K_B-C_Ux, Package_DFN_QFN:QFN-32-1EP_5x5mm_P0.5mm_EP3.45x3.45mm, symbol MCU_ST_STM32L4:STM32L431K_B-C_Ux
- renumbered U16 to U1
Connections:
- net A_HIGH2: now also U7.20 (PA10)
- net A_HIGH3: now also U10.20 (PA10)
- net A_HIGH4: now also U13.20 (PA10)
- net A_LOW2: now also U7.15 (PB1)
- net A_LOW3: now also U10.15 (PB1)
- net A_LOW4: now also U13.15 (PB1)
- net BEMF_A2: now also U7.6 (PA0)
- net BEMF_A3: now also U10.6 (PA0)
- net BEMF_A4: now also U13.6 (PA0)
- net BEMF_B2: now also U7.10 (PA4)
- net BEMF_B3: now also U10.10 (PA4)
- net BEMF_B4: now also U13.10 (PA4)
- net BEMF_C2: now also U7.11 (PA5)
- net BEMF_C3: now also U10.11 (PA5)
- net BEMF_C4: now also U13.11 (PA5)
- net BEMF_COMMON2: now also U7.7 (PA1)
- net BEMF_COMMON3: now also U10.7 (PA1)
- net BEMF_COMMON4: now also U13.7 (PA1)
- net B_HIGH2: now also U7.19 (PA9)
- net B_HIGH3: now also U10.19 (PA9)
- net B_HIGH4: now also U13.19 (PA9)
- net B_LOW2: now also U7.14 (PB0)
- net B_LOW3: now also U10.14 (PB0)
- net B_LOW4: now also U13.14 (PB0)
- net CURR2: now also U7.9 (PA3)
- net CURR3: now also U10.9 (PA3)
- net CURR4: now also U13.9 (PA3)
- net C_HIGH2: now also U7.18 (PA8)
- net C_HIGH3: now also U10.18 (PA8)
- net C_HIGH4: now also U13.18 (PA8)
- net C_LOW2: now also U7.13 (PA7)
- net C_LOW3: now also U10.13 (PA7)
- net C_LOW4: now also U13.13 (PA7)
- net SWDCLK2: now also U7.24 (PA14)
- net SWDCLK3: now also U10.24 (PA14)
- net SWDCLK4: now also U13.24 (PA14)
- net SWDIO2: now also U7.23 (PA13)
- net SWDIO3: now also U10.23 (PA13)
- net SWDIO4: now also U13.23 (PA13)
- net TELEMETRY: now also U10.29 (PB6), U13.29 (PB6), U7.29 (PB6)
- net TELEMRX: now also U10.30 (PB7), U13.30 (PB7), U7.30 (PB7)
- net VCC: now also U1.1 (VDD), U1.17 (VDD), U1.5 (VDDA), U10.1 (VDD), U10.17 (VDD), U10.5 (VDDA), U13.1 (VDD), U13.17 (VDD), U13.5 (VDDA), U7.1 (VDD), U7.17 (VDD), U7.5 (VDDA)
- net V_SENS2: now also U7.12 (PA6)
- net V_SENS3: now also U10.12 (PA6)
- net V_SENS4: now also U13.12 (PA6)
- net at R24.2: now also U7.27 (PB4)
- net at C23.1: now also U7.4 (NRST)
- net at R64.2: now also U13.27 (PB4)
- net at C37.1: now also U10.4 (NRST)
- net at C51.1: now also U13.4 (NRST)
- net at R44.2: now also U10.27 (PB4)
- new net: U10.16 (VSS), U10.32 (VSS), U10.33 (VSS)
- new net: U13.16 (VSS), U13.32 (VSS), U13.33 (VSS)
- new net: U7.16 (VSS), U7.32 (VSS), U7.33 (VSS)
- no-connect marks 85 -> 52
Other:
- moved on the sheet: C1, J5, J6, R1, R24, R44, R64, U1

Commit message: push
Parts:
- added C20, C34, C48, C72: 10u, Capacitor_SMD:C_1210_3225Metric, symbol Device:C
- added C7: 68uF, symbol Device:C_Polarized
Connections:
- net +9V: now also C20.1, C48.1, C7.1
- net +BATT: now also C15.1, U4.5 (EN), U4.7 (VIN)
- net GND: now also U10.16 (VSS), U10.32 (VSS), U10.33 (VSS), U13.16 (VSS), U13.32 (VSS), U13.33 (VSS), U7.16 (VSS), U7.32 (VSS), U7.33 (VSS), C20.2, C34.2, C48.2, C7.2, C72.2
- net VCC: now also C34.1, C72.1
Other:
- moved on the sheet: C15, C16, D4, D5, L1, R10, R11, R23, U4

Commit message: poush up to date
its been a long time since i last pushed but some updates were on the way
Parts:
- removed J4: Conn_01x08, Connector_JST:JST_SH_SM08B-SRSS-TB_1x08-1MP_P1.00mm_Horizontal, symbol Connector_Generic:Conn_01x08
- removed U4: TPS5430DDA, Package_SO:TI_SO-PowerPAD-8_ThermalVias, symbol Regulator_Switching:TPS5430DDA
- added J4: Conn_01x08_MountingPin, Connector_JST:JST_SH_SM08B-SRSS-TB_1x08-1MP_P1.00mm_Horizontal, symbol Connector_Generic_MountingPin:Conn_01x08_MountingPin
- added U4: LM76003, Package_DFN_QFN:Texas_RNP0030B_WQFN-30-1EP_4x6mm_P0.5mm_EP1.8x4.5mm_ThermalVias, symbol Regulator_Switching:LM76003
- C14, C15, C20, C24, C31, C34, C38, C4, C45, C48, C52, C59, C60, C61, C62, C63, C64, C65, C66, C67, C68, C69, C70, C72, C9: footprint Capacitor_SMD:C_1210_3225Metric -> Capacitor_SMD:C_0805_2012Metric
- C7: footprint (none) -> Capacitor_Tantalum_SMD:CP_EIA-6032-28_Kemet-C
- C71: footprint (none) -> Capacitor_THT:C_Disc_D5.0mm_W2.5mm_P5.00mm
- J1, J2, J21, J3: footprint (none) -> footprint_lib:Phase_Pads
- L1: footprint (none) -> Inductor_SMD:L_Chilisin_BMRF00101040
- Q1, Q10, Q11, Q12, Q13, Q14, Q15, Q16, Q17, Q18, Q19, Q2, Q20, Q21, Q22, Q23, Q24, Q3, Q4, Q5, Q6, Q7, Q8, Q9: footprint (none) -> easyeda2kicad:DFN-8_L5.8-W4.9-P1.27-LS6.0-BL-1
- R1, R10, R11, R12, R13, R14, R15, R16, R17, R18, R19, R20, R21, R22, R23, R24, R25, R26, R27, R28, R29, R3, R30, R31, R33, R34, R35, R36, R37, R38, R39, R4, R40, R41, R43, R44, R45, R46, R47, R48, R49, R5, R50, R53, R54, R55, R56, R57, R58, R59, R6, R60, R61, R63, R64, R65, R66, R67, R68, R69, R7, R70, R73, R74, R75, R76, R77, R78, R79, R8, R80, R81, R83, R9: footprint (none) -> Resistor_SMD:R_0402_1005Metric
- R2, R42, R62, R82: footprint (none) -> Resistor_SMD:R_2010_5025Metric
Connections:
- net +9V: no longer L1.2
- net +BATT: now also Q1.D, Q13.D, Q14.D, Q15.D, Q19.D, Q20.D, Q21.D, Q3.D, Q5.D, Q7.D, Q8.D, Q9.D; no longer Q1.1 (D), Q13.1 (D), Q14.1 (D), Q15.1 (D), Q19.1 (D), Q20.1 (D), Q21.1 (D), Q3.1 (D), Q5.1 (D), Q7.1 (D), Q8.1 (D), Q9.1 (D)
- net GND: now also U12.6 (REF2), U15.6 (REF2), U2.6 (REF2), U9.6 (REF2), J4.2 (Pin_2), J4.MP (MountPin), U4.19 (NC_{GND}), U4.24 (PGND), U4.25 (PGND), U4.26 (PGND), U4.29 (NC_{GND}); no longer C15.2, C7.2, R11.1
- net MOT_A1: now also Q1.S, Q2.D; no longer Q1.3 (S), Q10.1 (D), Q2.1 (D), Q7.3 (S)
- net MOT_A2: now also Q10.D, Q7.S
- net MOT_A3: now also Q13.S, Q16.D; no longer Q13.3 (S), Q16.1 (D)
- net MOT_A4: now also Q19.S, Q22.D; no longer Q19.3 (S), Q22.1 (D)
- net MOT_B1: now also Q3.S, Q4.D; no longer Q3.3 (S), Q4.1 (D)
- net MOT_B2: now also Q11.D, Q8.S; no longer Q11.1 (D), Q8.3 (S)
- net MOT_B3: now also Q14.S, Q17.D; no longer Q14.3 (S), Q17.1 (D)
- net MOT_B4: now also Q20.S, Q23.D; no longer Q20.3 (S), Q23.1 (D)
- net MOT_C1: now also Q5.S, Q6.D; no longer Q5.3 (S), Q6.1 (D)
- net MOT_C2: now also Q12.D, Q9.S; no longer Q12.1 (D), Q9.3 (S)
- net MOT_C3: now also Q15.S, Q18.D; no longer Q15.3 (S), Q18.1 (D)
- net MOT_C4: now also Q21.S, Q24.D; no longer Q21.3 (S), Q24.1 (D)
- net SIG_IN1: now also J4.5 (Pin_5)
- net SIG_IN2: now also J4.6 (Pin_6)
- net SIG_IN3: now also J4.7 (Pin_7)
- net SIG_IN4: now also J4.8 (Pin_8)
- net TELEMETRY: now also J4.4 (Pin_4)
- net TELEMRX: now also J4.3 (Pin_3)
- net VCC: no longer U12.6 (REF2), U15.6 (REF2), U2.6 (REF2), U9.6 (REF2)
- net at R81.1: now also Q24.G; no longer Q24.2 (G)
- net at R79.1: now also Q22.G; no longer Q22.2 (G)
- net at R38.1: now also Q9.G; no longer Q9.2 (G)
- net at R31.2: now also J4.1 (Pin_1)
- net at R57.1: now also Q14.G; no longer Q14.2 (G)
- net at R76.1: now also Q19.G; no longer Q19.2 (G)
- net at R9.1: now also Q6.G; no longer Q6.2 (G)
- net at R37.1: now also Q8.G; no longer Q8.2 (G)
- net at R5.1: now also Q2.G; no longer Q2.2 (G)
- net at C16.1: now also U4.6 (BOOT)
- net at C16.2, L1.1: now also U4.1 (SW), U4.2 (SW), U4.3 (SW), U4.4 (SW), U4.5 (SW); no longer D4.1 (K)
- net at R40.1: now also Q11.G; no longer Q11.2 (G)
- net at R4.1: now also Q1.G; no longer Q1.2 (G)
- net at R60.1: now also Q17.G; no longer Q17.2 (G)
- net at R77.1: now also Q20.G; no longer Q20.2 (G)
- net at R78.1: now also Q21.G; no longer Q21.2 (G)
- net at R39.1: now also Q10.G; no longer Q10.2 (G)
- net at R61.1: now also Q18.G; no longer Q18.2 (G)
- net at R56.1: now also Q13.G; no longer Q13.2 (G)
- net at R6.1: now also Q3.G; no longer Q3.2 (G)
- net at R7.1: now also Q4.G; no longer Q4.2 (G)
- net at R41.1: now also Q12.G; no longer Q12.2 (G)
- net at R36.1: now also Q7.G; no longer Q7.2 (G)
- net at R8.1: now also Q5.G; no longer Q5.2 (G)
- net at R58.1: now also Q15.G; no longer Q15.2 (G)
- net at R59.1: now also Q16.G; no longer Q16.2 (G)
- net at R80.1: now also Q23.G; no longer Q23.2 (G)
- new net: Q16.S, Q17.S, Q18.S, R62.1, U12.2 (+)
- new net: Q2.S, Q4.S, Q6.S, R2.1, U2.2 (+)
- new net: Q10.S, Q11.S, Q12.S, R42.1, U9.2 (+)
- new net: Q22.S, Q23.S, Q24.S, R82.1, U15.2 (+)
- new net: L1.2, U4.9 (BIAS)
- new net: U4.13 (AGND), U4.14 (AGND), U4.15 (AGND), U4.31 (AGND)
- new net: U4.20 (PVIN), U4.21 (PVIN), U4.22 (PVIN)
- new net: C15.2, C7.2, R11.1
Other:
- moved on the sheet: C16, L1, R21, R22

Commit message: wip
Parts:
- removed C29, C43: 100n, Capacitor_SMD:C_0402_1005Metric, symbol Device:C
- removed C48, C72: 10u, Capacitor_SMD:C_0805_2012Metric, symbol Device:C
- removed C7: 68uF, Capacitor_Tantalum_SMD:CP_EIA-6032-28_Kemet-C, symbol Device:C_Polarized
- removed D4: SS26, Diode_SMD:D_SMA, symbol Diode:SS26
- removed U12, U15, U2, U9: INA240A1PW, Package_SO:TSSOP-8_4.4x3mm_P0.65mm, symbol Amplifier_Current:INA240A1PW
- removed U5, U6: AMS1117-3.3, Package_TO_SOT_SMD:SOT-223-3_TabPin2, symbol Regulator_Linear:AMS1117-3.3
- added C73: 1u, Capacitor_SMD:C_0402_1005Metric, symbol Device:C
- added C74: 2.2u, Capacitor_SMD:C_0402_1005Metric, symbol Device:C
- added C75: 100n, Capacitor_SMD:C_0402_1005Metric, symbol Device:C
- added C76: 2.2u, Capacitor_SMD:C_0603_1608Metric, symbol Device:C
- added C77: 5.1p, Capacitor_SMD:C_0402_1005Metric, symbol Device:C
- added C78, C79: 10u, Capacitor_SMD:C_0805_2012Metric, symbol Device:C
- added R32: 105k, Resistor_SMD:R_0402_1005Metric, symbol Device:R
- added R51: 36.5k, Resistor_SMD:R_0402_1005Metric, symbol Device:R
- added R71, R72, R84, R85: 10k, Resistor_SMD:R_0402_1005Metric, symbol Device:R
- added U2: INA4180A2, Package_SO:TSSOP-14_4.4x5mm_P0.65mm, symbol Amplifier_Current:INA4180A2
- added U5: LDL212PV33R, easyeda2kicad:DFN-6_L2.0-W2.0-P0.50-BL-EP1.45, symbol easyeda2kicad:LDL212PV33R
- C16: value 10n -> 470n; LCSC C15195 -> C92361
- D1, D10, D11, D12, D13, D14, D2, D3, D6, D7, D8, D9: value 1N4148W -> 1N4148WT; footprint Diode_SMD:D_SOD-123 -> Diode_SMD:D_SOD-523
- J10, J11, J12, J5, J6, J7, J8, J9: footprint TestPoint:TestPoint_Pad_1.0x1.0mm -> TestPoint:TestPoint_Pad_D1.0mm
- L1: footprint Inductor_SMD:L_Chilisin_BMRF00101040 -> footprint_lib:inductor FANGCHENG FC-ALX 5050D-150MT; LCSC (none) -> C5370912
- Q1, Q10, Q11, Q12, Q13, Q14, Q15, Q16, Q17, Q18, Q19, Q2, Q20, Q21, Q22, Q23, Q24, Q3, Q4, Q5, Q6, Q7, Q8, Q9: value NMOS -> RS60N80UHG; LCSC (none) -> C51904706
- R10: value 10k -> 100k
- R11: value 1.58k -> 12.4k
- R2, R42, R62, R82: value 2mr -> 1mr; footprint Resistor_SMD:R_2010_5025Metric -> Resistor_SMD:R_1210_3225Metric; LCSC (none) -> C4173351
- U1, U10, U13, U7: value STM32L431K_B-C_Ux -> STM32F051K8U6; LCSC (none) -> C72339
- U4: value LM76003 -> LM76003/2; LCSC (none) -> C470958
Connections:
- net V_SENS1 is gone; now on net V_SENS: U1.12 (PA6)
- net V_SENS2 is gone; now on net V_SENS: U7.12 (PA6)
- net V_SENS3 is gone; now on net V_SENS: U10.12 (PA6)
- net V_SENS4 is gone; now on net V_SENS: U13.12 (PA6)
- net +9V: now also L1.2, U4.9 (BIAS), C73.1, C75.1, C77.2, C78.1, C79.1, R32.1, U5.4 (VIN), U5.6 (EN)
- net +BATT: now also U4.18 (EN), U4.20 (PVIN), U4.21 (PVIN), U4.22 (PVIN), C76.1
- net GND: now also C15.2, R11.1, U4.13 (AGND), U4.14 (AGND), U4.15 (AGND), U4.17 (SYNC/MODE), U4.27 (NC_{GND}), U4.28 (NC_{GND}), U4.30 (NC_{GND}), U4.31 (AGND), C73.2, C74.2, C75.2, C76.2, C78.2, C79.2, R51.2, R71.1, R72.1, R84.1, R85.1, U2.11 (GND), U5.1 (GND), U5.7 (EP); no longer R2.2, R42.2, R62.2, R82.2
- net VCC: now also U2.4 (VS), U5.2 (ADJ/sense), U5.3 (VOUT)
- net curr3+: now reaches Q16.S, Q17.S, Q18.S, R62.1
- net curr3+: now also U2.12 (+)
- net curr1+: now reaches Q2.S, Q4.S, Q6.S, R2.1
- net curr1+: now also U2.10 (+)
- net at R10.1, R11.2: now also U4.12 (FB), C77.1
- net curr2+: now reaches Q10.S, Q11.S, Q12.S, R42.1
- net curr2+: now also U2.5 (+)
- net at R43.1: now also U2.7
- net at R3.1: now also U2.8
- net at U10.31 (PH3): now also R72.2
- net at U13.31 (PH3): now also R71.2
- net at R83.1: now also U2.1
- net curr4+: now reaches Q22.S, Q23.S, Q24.S, R82.1
- net curr4+: now also U2.3 (+)
- net at U1.31 (PH3): now also R85.2
- net at U4.10 (RT): now also R51.1
- net at U4.16 (PGOOD): now also R32.2
- net at U4.8 (VCC): now also C74.1
- net at U7.31 (PH3): now also R84.2
- net at R63.1: now also U2.14
- new net curr1-: R2.2, U2.9 (-)
- new net curr2-: R42.2, U2.6 (-)
- new net curr3-: R62.2, U2.13 (-)
- new net curr4-: R82.2, U2.2 (-)
- no-connect marks 52 -> 49
Other:
- moved on the sheet: C1, C15, C16, C17, C20, C30, C34, C44, C57, C58, C8, D5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

Commit message: a
Parts:
- removed C1, C10, C17, C18, C19, C22, C23, C25, C3, C32, C33, C36, C37, C39, C46, C47, C5, C50, C51, C53, C57, C6, C75: 100n, Capacitor_SMD:C_0402_1005Metric, symbol Device:C
- removed C11, C12, C13, C2, C21, C26, C27, C28, C35, C40, C41, C42, C49, C54, C55, C56: 1u, Capacitor_SMD:C_0603_1608Metric, symbol Device:C
- removed C14, C15, C20, C24, C31, C34, C38, C4, C45, C52, C59, C60, C61, C62, C63, C64, C65, C66, C67, C68, C69, C70, C78, C79, C9: 10u, Capacitor_SMD:C_0805_2012Metric, symbol Device:C
- removed C16: 470n, Capacitor_SMD:C_0402_1005Metric, symbol Device:C
- removed C30, C44, C58, C8: 10n, Capacitor_SMD:C_0402_1005Metric, symbol Device:C
- removed C71: C_Polarized, Capacitor_THT:C_Disc_D5.0mm_W2.5mm_P5.00mm, symbol Device:C_Polarized
- removed C73: 1u, Capacitor_SMD:C_0402_1005Metric, symbol Device:C
- removed C74: 2.2u, Capacitor_SMD:C_0402_1005Metric, symbol Device:C
- removed C76: 2.2u, Capacitor_SMD:C_0603_1608Metric, symbol Device:C
- removed C77: 5.1p, Capacitor_SMD:C_0402_1005Metric, symbol Device:C
- removed D1, D10, D11, D12, D13, D14, D2, D3, D6, D7, D8, D9: 1N4148WT, Diode_SMD:D_SOD-523, symbol Diode:1N4148W
- removed D15: SMBJ28A, Diode_SMD:D_SMB, symbol Diode:SM6T27A
- removed D5: LED, Diode_SMD:D_0603_1608Metric, symbol Device:LED
- removed J1, J2, J21, J3: Conn_01x03, footprint_lib:Phase_Pads, symbol Connector_Generic:Conn_01x03
- removed J10, J11, J12, J5, J6, J7, J8, J9: Conn_01x01, TestPoint:TestPoint_Pad_D1.0mm, symbol Connector_Generic:Conn_01x01
- removed J4: Conn_01x08_MountingPin, Connector_JST:JST_SH_SM08B-SRSS-TB_1x08-1MP_P1.00mm_Horizontal, symbol Connector_Generic_MountingPin:Conn_01x08_MountingPin
- removed L1: 100u, footprint_lib:inductor FANGCHENG FC-ALX 5050D-150MT, symbol Device:L
- removed Q1, Q10, Q11, Q12, Q13, Q14, Q15, Q16, Q17, Q18, Q19, Q2, Q20, Q21, Q22, Q23, Q24, Q3, Q4, Q5, Q6, Q7, Q8, Q9: RS60N80UHG, easyeda2kicad:DFN-8_L5.8-W4.9-P1.27-LS6.0-BL-1, symbol Simulation_SPICE:NMOS
- removed R1, R12, R17, R20, R23, R24, R3, R33, R34, R35, R43, R44, R53, R54, R55, R63, R64, R73, R74, R75, R83: 1k, Resistor_SMD:R_0402_1005Metric, symbol Device:R
- removed R10, R21: 100k, Resistor_SMD:R_0402_1005Metric, symbol Device:R
- removed R11: 12.4k, Resistor_SMD:R_0402_1005Metric, symbol Device:R
- removed R13, R14, R15, R16, R18, R19, R22, R25, R26, R27, R28, R29, R30, R45, R46, R47, R48, R49, R50, R65, R66, R67, R68, R69, R70, R71, R72, R84, R85: 10k, Resistor_SMD:R_0402_1005Metric, symbol Device:R
- removed R2, R42, R62, R82: 1mr, Resistor_SMD:R_1210_3225Metric, symbol Device:R
- removed R31: 0r, Resistor_SMD:R_0402_1005Metric, symbol Device:R
- removed R32: 105k, Resistor_SMD:R_0402_1005Metric, symbol Device:R
- removed R36, R37, R38, R39, R4, R40, R41, R5, R56, R57, R58, R59, R6, R60, R61, R7, R76, R77, R78, R79, R8, R80, R81, R9: 20r, Resistor_SMD:R_0402_1005Metric, symbol Device:R
- removed R51: 36.5k, Resistor_SMD:R_0402_1005Metric, symbol Device:R
- removed U1, U10, U13, U7: STM32F051K8U6, Package_DFN_QFN:QFN-32-1EP_5x5mm_P0.5mm_EP3.45x3.45mm, symbol MCU_ST_STM32L4:STM32L431K_B-C_Ux
- removed U11, U14, U3, U8: FD6288Q_C328453, easyeda2kicad:QFN-24_L4.0-W4.0-P0.50-BL-EP2.6, symbol easyeda2kicad:FD6288Q_C328453
- removed U2: INA4180A2, Package_SO:TSSOP-14_4.4x5mm_P0.65mm, symbol Amplifier_Current:INA4180A2
- removed U4: LM76003/2, Package_DFN_QFN:Texas_RNP0030B_WQFN-30-1EP_4x6mm_P0.5mm_EP1.8x4.5mm_ThermalVias, symbol Regulator_Switching:LM76003
- removed U5: LDL212PV33R, easyeda2kicad:DFN-6_L2.0-W2.0-P0.50-BL-EP1.45, symbol easyeda2kicad:LDL212PV33R
- added J13, J14, J19, J20, J27, J28: Conn_02x05_Odd_Even, Connector_PinHeader_1.00mm:PinHeader_2x05_P1.00mm_Vertical, symbol Connector_Generic:Conn_02x05_Odd_Even
- added J15: Conn_02x07_Odd_Even, Connector_PinHeader_1.00mm:PinHeader_2x07_P1.00mm_Vertical, symbol Connector_Generic:Conn_02x07_Odd_Even
- added J16, J17, J18, J22, J23, J24, J25, J26: Conn_01x02, Connector_PinHeader_1.00mm:PinHeader_1x02_P1.00mm_Vertical, symbol Connector_Generic:Conn_01x02
- added J29: Conn_02x04_Odd_Even, Connector_PinHeader_1.00mm:PinHeader_2x04_P1.00mm_Vertical, symbol Connector_Generic:Conn_02x04_Odd_Even
Connections:
- net +9V: now also J15.10 (Pin_10), J15.6 (Pin_6), J29.6 (Pin_6)
- net GND: now also J13.7 (Pin_7), J14.3 (Pin_3), J15.7 (Pin_7), J19.3 (Pin_3), J20.7 (Pin_7), J27.7 (Pin_7), J28.3 (Pin_3), J29.7 (Pin_7)
- net VCC: now also J15.5 (Pin_5), J15.9 (Pin_9), J29.5 (Pin_5)
- new net Powerstage/GHA1: J27.10 (Pin_10)
- new net Powerstage/GHA2: J28.4 (Pin_4)
- new net Powerstage/GHA3: J19.2 (Pin_2)
- new net Powerstage/GHA4: J20.8 (Pin_8)
- new net Powerstage/GHB1: J27.2 (Pin_2)
- new net Powerstage/GHB2: J28.8 (Pin_8)
- new net Powerstage/GHB3: J19.10 (Pin_10)
- new net Powerstage/GHB4: J20.4 (Pin_4)
- new net Powerstage/GHC1: J27.3 (Pin_3)
- new net Powerstage/GHC2: J28.5 (Pin_5)
- new net Powerstage/GHC3: J19.7 (Pin_7)
- new net Powerstage/GHC4: J20.5 (Pin_5)
- new net Powerstage/GLA1: J27.9 (Pin_9)
- new net Powerstage/GLA2: J28.2 (Pin_2)
- new net Powerstage/GLA3: J19.1 (Pin_1)
- new net Powerstage/GLA4: J20.10 (Pin_10)
- new net Powerstage/GLB1: J27.6 (Pin_6)
- new net Powerstage/GLB2: J28.10 (Pin_10)
- new net Powerstage/GLB3: J19.6 (Pin_6)
- new net Powerstage/GLB4: J20.2 (Pin_2)
- new net Powerstage/GLC1: J27.1 (Pin_1)
- new net Powerstage/GLC2: J28.9 (Pin_9)
- new net Powerstage/GLC3: J19.9 (Pin_9)
- new net Powerstage/GLC4: J20.1 (Pin_1)
- new net Powerstage/MOT_A1: J27.8 (Pin_8)
- new net Powerstage/MOT_A2: J28.1 (Pin_1)
- new net Powerstage/MOT_A3: J19.4 (Pin_4)
- new net Powerstage/MOT_A4: J20.9 (Pin_9)
- new net Powerstage/MOT_B1: J27.4 (Pin_4)
- new net Powerstage/MOT_B2: J28.6 (Pin_6)
- new net Powerstage/MOT_B3: J19.8 (Pin_8)
- new net Powerstage/MOT_B4: J20.6 (Pin_6)
- new net Powerstage/MOT_C1: J27.5 (Pin_5)
- new net Powerstage/MOT_C2: J28.7 (Pin_7)
- new net Powerstage/MOT_C3: J19.5 (Pin_5)
- new net Powerstage/MOT_C4: J20.3 (Pin_3)
- new net Powerstage/SIG_IN1: J15.13 (Pin_13)
- new net Powerstage/SIG_IN2: J15.14 (Pin_14)
- new net Powerstage/SIG_IN3: J15.2 (Pin_2)
- new net Powerstage/SIG_IN4: J15.1 (Pin_1)
- new net Powerstage/TELEMETRY: J15.11 (Pin_11), J15.3 (Pin_3)
- new net Powerstage/TELEMRX: J15.12 (Pin_12), J15.4 (Pin_4)
- new net Powerstage/V_SENS: J15.8 (Pin_8)
- new net Powerstage/curr1+: J22.2 (Pin_2)
- new net Powerstage/curr1-: J22.1 (Pin_1)
- new net Powerstage/curr2+: J18.2 (Pin_2)
- new net Powerstage/curr2-: J18.1 (Pin_1)
- new net Powerstage/curr3+: J16.2 (Pin_2)
- new net Powerstage/curr3-: J16.1 (Pin_1)
- new net Powerstage/curr4+: J17.2 (Pin_2)
- new net Powerstage/curr4-: J17.1 (Pin_1)
- new net bottom/GHA3: J14.2 (Pin_2)
- new net bottom/GHA4: J13.8 (Pin_8)
- new net bottom/GHB3: J14.10 (Pin_10)
- new net bottom/GHB4: J13.4 (Pin_4)
- new net bottom/GHC3: J14.7 (Pin_7)
- new net bottom/GHC4: J13.5 (Pin_5)
- new net bottom/GLA3: J14.1 (Pin_1)
- new net bottom/GLA4: J13.10 (Pin_10)
- new net bottom/GLB3: J14.6 (Pin_6)
- new net bottom/GLB4: J13.2 (Pin_2)
- new net bottom/GLC3: J14.9 (Pin_9)
- new net bottom/GLC4: J13.1 (Pin_1)
- new net bottom/MOT_A3: J14.4 (Pin_4)
- new net bottom/MOT_A4: J13.9 (Pin_9)
- new net bottom/MOT_B3: J14.8 (Pin_8)
- new net bottom/MOT_B4: J13.6 (Pin_6)
- new net bottom/MOT_C3: J14.5 (Pin_5)
- new net bottom/MOT_C4: J13.3 (Pin_3)
- new net bottom/SIG_IN3: J29.1 (Pin_1)
- new net bottom/SIG_IN4: J29.2 (Pin_2)
- new net bottom/TELEMETRY: J29.3 (Pin_3)
- new net bottom/TELEMRX: J29.4 (Pin_4)
- new net bottom/V_SENS: J29.8 (Pin_8)
- new net bottom/curr3+: J26.1 (Pin_1)
- new net bottom/curr3-: J26.2 (Pin_2)
- new net bottom/curr4+: J25.2 (Pin_2)
- new net bottom/curr4-: J25.1 (Pin_1)
- new net top/curr1+: J23.2 (Pin_2)
- new net top/curr1-: J23.1 (Pin_1)
- new net top/curr2+: J24.2 (Pin_2)
- new net top/curr2-: J24.1 (Pin_1)
- no-connect marks 49 -> 0
Other:
- added sheet Powerstage (pow.kicad_sch)
- added sheet bottom (bottom.kicad_sch)
- added sheet top (top.kicad_sch)
- note removed: "BEMF Sensing Resistor Network"
- note removed: "Gate drivers"
- note removed: "MCU"
- note removed: "Motor phase"
- note removed: "NOTE: repurposed BATT_CURR with TELEMRX for firmware update to esc since we have individual shunts per esc"
- note removed: "Powerstage and Current sensing"
- note removed: "Voltage regulators"
- note removed: "betaflight "standardized" connector"
- note removed: "caps and protection"

Commit message: a
Other:
- sheet bottom ports: added 9v; removed none
Changed lines of the file:
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@@
 		(color 0 0 0 0)
 	)
+	(junction
+		(at 170.18 177.8)
+		(diameter 0)
+		(color 0 0 0 0)
+	)
 	(wire
 		(pts
@@
 	(wire
 		(pts
+			(xy 171.45 187.96) (xy 171.45 177.8)
+		)
+		(stroke
+			(width 0)
+			(type default)
+		)
+	)
+	(wire
+		(pts
 			(xy 200.66 87.63) (xy 146.05 87.63)
 		)
@@
 	(wire
 		(pts
+			(xy 170.18 177.8) (xy 171.45 177.8)
+		)
+		(stroke
+			(width 0)
+			(type default)
+		)
+	)
+	(wire
+		(pts
 			(xy 82.55 39.37) (xy 95.25 39.37)
 		)
@@
 	(wire
 		(pts
+			(xy 132.08 187.96) (xy 171.45 187.96)
+		)
+		(stroke
+			(width 0)
+			(type default)
+		)
+	)
+	(wire
+		(pts
 			(xy 91.44 161.29) (xy 91.44 167.64)
 		)
@@
 	(wire
 		(pts
+			(xy 132.08 181.61) (xy 132.08 187.96)
+		)
+		(stroke
+			(width 0)
+			(type default)
+		)
+	)
+	(wire
+		(pts
 			(xy 66.04 39.37) (xy 57.15 39.37)
 		)
@@
 			(effects
 				(font
+					(size 1.27 1.27)
+				)
+				(justify left)
+			)
+		)
+		(pin "9v" bidirectional
+			(at 132.08 181.61 270)
+			(effects
+				(font
