File: src/hardware/esc/pow.kicad_sch (KiCad schematic)
At the start: 94 parts, among them J1 Conn_01x03, J2 Conn_01x03, J21 Conn_01x03, J3 Conn_01x03, J4 Conn_01x08_MountingPin, Q1 RS60N80UHG, Q10 RS60N80UHG, Q11 RS60N80UHG, Q12 RS60N80UHG, Q13 RS60N80UHG, Q14 RS60N80UHG, Q15 RS60N80UHG, Q16 RS60N80UHG, Q17 RS60N80UHG, Q18 RS60N80UHG, Q19 RS60N80UHG, Q2 RS60N80UHG, Q20 RS60N80UHG, Q21 RS60N80UHG, Q22 RS60N80UHG, Q23 RS60N80UHG, Q24 RS60N80UHG, Q3 RS60N80UHG, Q4 RS60N80UHG, Q5 RS60N80UHG, Q6 RS60N80UHG, Q7 RS60N80UHG, Q8 RS60N80UHG, Q9 RS60N80UHG, U4 LM76003/2, U5 LDL212PV33R

Commit message: a
Parts:
- C15, C20, C34, C59, C60, C61, C62, C63, C64, C65, C66, C67, C68, C69, C70: LCSC C13585 -> C3039694
- C71, J1, J2, J21, J3: LCSC (none) -> x; now left out of the parts list
- C73: LCSC (none) -> C913556
- C74: LCSC (none) -> C12530
- C76: LCSC C415535 -> C913904
- D15: LCSC (none) -> C178227
- D5: LCSC (none) -> C7496819
- J4: LCSC (none) -> C160407
- R10, R21: LCSC (none) -> C445619
- R11: LCSC (none) -> C490814
- R22: LCSC (none) -> C190095
- R23: LCSC (none) -> C445596
- R31: LCSC (none) -> x(shunt); now left out of the parts list
- R32: LCSC (none) -> C2933067
- R36, R37, R38, R39, R4, R40, R41, R5, R56, R57, R58, R59, R6, R60, R61, R7, R76, R77, R78, R79, R8, R80, R81, R9: LCSC (none) -> C2909334
- R51: LCSC (none) -> C42396638
- U5: LCSC (none) -> C2969892
