File: src/hardware/esc/top.kicad_sch (KiCad schematic)
At the start: 64 parts, among them J5 Conn_01x01, J6 Conn_01x01, J7 Conn_01x01, J8 Conn_01x01, U1 STM32F051K8U6, U2 INA2180A1, U3 FD6288Q_C328453, U7 STM32F051K8U6, U8 FD6288Q_C328453

Commit message: a
Changed lines of the file:
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@@
+	(wire
+		(pts
+			(xy 229.87 22.86) (xy 223.52 22.86)
+		)
+		(stroke
+			(width 0)
+			(type default)
+		)
+	)
 	(wire
 		(pts
@@
 	(label "vcc"
 		(at 146.05 158.75 0)
+		(effects
+			(font
+				(size 1.27 1.27)
+			)
+			(justify left bottom)
+		)
+	)
+	(label "9v"
+		(at 229.87 22.86 0)
 		(effects
 			(font
@@
 		)
 	)
+	(hierarchical_label "9v"
+		(shape bidirectional)
+		(at 223.52 22.86 180)
+		(effects
+			(font
+				(size 1.27 1.27)
+			)
+			(justify right)
+		)
+	)

Commit message: a
Parts:
- C14, C4: LCSC C13585 -> C3039694
- C24, C9: LCSC (none) -> C962136
- D1, D2, D3, D6, D7, D8: LCSC (none) -> C917006
- J5, J6, J7, J8: LCSC (none) -> x
- R1, R12, R17, R20, R24, R3, R33, R34, R35, R43: LCSC (none) -> C445596
- R13, R14, R15, R16, R18, R19, R25, R26, R27, R28, R29, R30, R84, R85: LCSC (none) -> C190095
- U2: LCSC (none) -> C2873353
